File: Small_load_V1/Small_load_V1.kicad_sch (KiCad schematic)
At the start: 10 parts

Commit message: v
Parts:
- removed J?: USB3_B, symbol Connector:USB3_B
- added FB1: FerriteBead_Small, symbol Device:FerriteBead_Small
- added H1, H2, H3, H4: M3, MountingHole:MountingHole_3.2mm_M3_Pad_TopBottom, symbol Mechanical:MountingHole_Pad
- added J1: USB_B, symbol Connector:USB_B
- added J2: Screw_Terminal_01x02, symbol Connector:Screw_Terminal_01x02
- added J3: Conn_01x02, Connector_PinSocket_2.54mm:PinSocket_1x02_P2.54mm_Vertical, symbol Connector_Generic:Conn_01x02
- added Q1: IRFZ24NPBF, Package_TO_SOT_THT:TO-220-3_Vertical, symbol Device:Q_NMOS_GDS
- added R2, R4: 1R, Resistor_THT:R_Axial_Power_L50.0mm_W9.0mm_P55.88mm, symbol Device:R_Small
- added R3: 10k, symbol Device:R_Small
- added U1: D1213A-02SM, Package_TO_SOT_SMD:SOT-23-5_HandSoldering, symbol My_custom_lib:D1213A-02SM
- HS1: renamed from HS?; footprint (none) -> Heatsink:Heatsink_Fischer_SK104-STCB_35x13mm__2xDrill3.5mm_ScrewM3
- gave numbers to parts that had none: 8
Connections:
- net GND: now also U3.2 (-), H1.1, H2.1, H3.1, H4.1, J1.4 (GND), J2.2 (Pin_2), R2.2, R3.1, R4.2, U1.2 (VSS)
- net +BATT: now reaches U3.1 (+)
- new net: J2.1 (Pin_1), Q1.2 (D)
- new net: J3.1 (Pin_1), Q1.3 (S), R2.1
- new net: J3.2 (Pin_2), R4.1
- new net +5V: FB1.1, U1.5 (VCC)
- new net D+: J1.3 (D+), U1.3 (CH1)
- new net D-: J1.2 (D-), U1.4 (CH2)
- new net VBUS: FB1.2, J1.1 (VBUS)
- no-connect marks 3 -> 5
Other:
- moved on the sheet: HS1

Commit message: Update Small_load_V1.kicad_sch
Parts:
- added U?: LM4040DBZ-2.0, Package_TO_SOT_SMD:SOT-23, symbol Reference_Voltage:LM4040DBZ-2.0
Changed lines of the file:
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@@
     (pin "1")
+  )
+  (symbol (lib_id "Reference_Voltage:LM4040DBZ-2.0") (at 97.79 40.64 0) (unit 1)
+    (in_bom yes) (on_board yes) (fields_autoplaced)
+    (property "Reference" "U?" (id 0) (at 97.79 34.29 0))
+    (property "Value" "LM4040DBZ-2.0" (id 1) (at 97.79 36.83 0))
+    (property "Footprint" "Package_TO_SOT_SMD:SOT-23" (id 2) (at 97.79 45.72 0)
+      (effects (font (size 1.27 1.27) italic) hide)
+    )
+    (property "Datasheet" "http://www.ti.com/lit/ds/symlink/lm4040-n.pdf" (id 3) (at 97.79 40.64 0)
+      (effects (font (size 1.27 1.27) italic) hide)
+    )
+    (pin "1")
+    (pin "2")
   )
   (symbol (lib_id "power:+BATT") (at 55.88 152.4 0) (unit 1)
@@
       (reference "U3") (unit 1) (value "1043") (footprint "1043")
     )
-  )
+    (path "/a5b2aaf7-e7a8-4469-a5a5-93c4786dc2c1"
+      (reference "U?") (unit 1) (value "LM4040DBZ-2.0") (footprint "Package_TO_SOT_SMD:SOT-23")
+    )
+  )

Commit message: f
Parts:
- added J4: Conn_02x04_Odd_Even, Connector_PinHeader_2.54mm:PinHeader_2x04_P2.54mm_Vertical, symbol Connector_Generic:Conn_02x04_Odd_Even
- added J?: Conn_01x03, Connector_PinHeader_2.54mm:PinHeader_1x03_P2.54mm_Vertical, symbol Connector_Generic:Conn_01x03
- added R5, R6: 65k, symbol Device:R_Small
- added R7: X, Resistor_THT:R_Axial_DIN0207_L6.3mm_D2.5mm_P10.16mm_Horizontal, symbol Device:R_Small
- added R8, R9: 10k, symbol Device:R_Small
- added TP?: TestPoint, TestPoint:TestPoint_Pad_D2.0mm, symbol Connector:TestPoint
- gave numbers to parts that had none: 1
Connections:
- net GND: now also J?.2 (Pin_2), R9.1
- net LOAD: now reaches J2.1 (Pin_1), Q1.2 (D)
- net LOAD: now also R5.1, R6.2, R7.2, R8.1
- net SPI_SS: now reaches U2.10 (PA4)
- net SPI_CLK: now reaches U2.11 (PA5)
- net SPI_MOSI: now reaches U2.12 (PA6)
- net SPI_MISO: now reaches U2.13 (PA7)
- net ADC_IN8: now reaches U2.14 (PB0)
- net ADC_REF: now reaches U2.15 (PB1)
- net Crystal_Clock_out: now reaches U2.18 (PA8)
- net Crystal_Clock_out: now also TP?.1
- net I2C_CLK: now reaches U2.19 (PA9)
- net I2C_SDA: now reaches U2.20 (PA10)
- net SWD_DIO: now reaches U2.23 (PA13)
- net SWD_DIO: now also J?.3 (Pin_3)
- net SWD_CLK: now reaches U2.24 (PA14)
- net SWD_CLK: now also J?.1 (Pin_1)
- net CLOCK_in: now reaches U2.6 (PA0)
- net ADC_IN1: now reaches U2.7 (PA1)
- net SYS_wakeup3: now reaches U2.8 (PA2)
- net ADC_IN3: now reaches U2.9 (PA3)
- new net: J4.4 (Pin_4), R5.2
- new net: J4.1 (Pin_1), J4.3 (Pin_3), J4.5 (Pin_5), J4.7 (Pin_7), R9.2
- new net: J4.2 (Pin_2), R7.1
- new net: J4.6 (Pin_6), R6.1
- new net: J4.8 (Pin_8), R8.2
Other:
- note added: "18650 cell holder"
- note added: "Absolute max voltage: 55V"
- note added: "Max voltage: 2V"
- note added: "THT custom"
- note added: "from left to right:"
- note added: "max voltage 55V"
- note added: "normal 12-15V line"
- moved on the sheet: HS1, J2, J3, Q1, R2, R3, R4, U3

Commit message: b
Parts:
- added C5, C6, C? (x2): 4u7, symbol Device:C_Small
- added C? (x3): 47n, symbol Device:C_Small
- added C? (x2): 1u, symbol Device:C_Small
- added D1, D? (x4): D_Small, symbol Device:D_Small
- added J6: Fan, symbol Connector_Generic:Conn_01x02
- added L1: 10uH, symbol Device:L
- added R11: 47k, symbol Device:R_Small
- added R12, R?: 100k, symbol Device:R_Small
- added R13: 5k1, symbol Device:R_Small
- added R? (x3): 1k, symbol Device:R_Small
- added R?: 20k, symbol Device:R_Small
- added R?: 100, symbol Device:R_Small
- added R?: 10k, symbol Device:R_Small
- added U5: 1602_LCD_I2C, Z_mycustom_footprint_lib:1602 LCD I2C, symbol My_custom_lib:1602_LCD_I2C
- added U6: LM324A, symbol Amplifier_Operational:LM324A
- added U8: AP3012KTR-G1, Package_TO_SOT_SMD:SOT-23-5_HandSoldering, symbol My_custom_lib:AP3012KTR-G1
- J1: footprint (none) -> Connector_USB:USB_A_CONNFLY_DS1095-WNR0
- J3: renamed from J2; footprint (none) -> TerminalBlock:TerminalBlock_Altech_AK300-2_P5.00mm
- gave numbers to parts that had none: 2
- renumbered J3 to J4, J4 to J5, R9 to R10, R5 to R4, R6 to R5, R2 to R6, R4 to R7, R7 to R8, R8 to R9, U3 to U1, U1 to U2, U4 to U3, U2 to U4
Connections:
- net +3V3: now also C6.1, U8.5 (Vin)
- net D+: now also U2.4 (CH2); no longer U2.3 (CH1)
- net D-: now also U2.3 (CH1); no longer U2.4 (CH2)
- net GND: now also C5.2, C6.2, C?.2, C?.2, C?.2, C?.2, C?.2, D?.1 (K), J6.1 (Pin_1), R12.2, R13.2, R?.1, R?.1, U8.2 (GND); no longer R3.1
- net I2C_CLK: now also U5.54 (SCL)
- net I2C_SDA: now also U5.53 (SDA)
- net LOAD_VOLTAGE: now also J5.1 (Pin_1), J5.3 (Pin_3), J5.5 (Pin_5), J5.7 (Pin_7), R10.2
- net PWM_SIGNAL1: now also R?.1
- net at Q1.1 (G): now also R?.2
- net at J4.1 (Pin_1), Q1.3 (S), R6.1: now also R3.1
- new net: C?.1, R?.2, U6.12 (+)
- new net: R?.1, R?.2, U6.9 (-)
- new net: R?.1, R?.2, U6.8
- new net: R?.1, U6.13 (-), U6.14
- new net: C?.1, R?.2, U6.10 (+)
- new net: C?.2, C?.2, L1.1, U8.1 (SW)
- new net: D1.2 (A), L1.2
- new net: C?.1, R?.2, U6.5 (+)
- new net: R?.1, R?.2, U6.6 (-), U6.7
- new net: C?.1, D?.1 (K), D?.2 (A) (x3)
- new net: U6.1, U6.2 (-)
- new net: R11.2, R13.1, U8.3 (FB)
- new net: R12.1, U8.4 (SHDN)
- new net +12V: C5.1, D1.1 (K), J6.2 (Pin_2), R11.1
- new net -3V3: C?.1, D?.2 (A)
- no-connect marks 5 -> 7
Other:
- note added: "12.77V"
- moved on the sheet: HS1, J2, J3, J4, J5, Q1, R1, R10, R4, R5, R6, R7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

Commit message: ;
Parts:
- removed C? (x2): 4u7, symbol Device:C_Small
- removed C? (x2): 1u, symbol Device:C_Small
- removed D? (x4): D_Small, symbol Device:D_Small
- added C10, C14, C18, C22: 100n, symbol Device:C_Small
- added C11, C?: 47u, Capacitor_THT:CP_Radial_D6.3mm_P2.50mm, symbol Device:C_Small
- added C13: 47n, symbol Device:C_Small
- added C15, C16, C17: 22u, Capacitor_SMD:C_0805_2012Metric_Pad1.18x1.45mm_HandSolder, symbol Device:C_Small
- added C19: 100n, Capacitor_SMD:C_0603_1608Metric_Pad1.08x0.95mm_HandSolder, symbol Device:C_Small
- added C20: 1u, Capacitor_SMD:C_0603_1608Metric_Pad1.08x0.95mm_HandSolder, symbol Device:C_Small
- added C21: 4.7u, Capacitor_SMD:C_0603_1608Metric_Pad1.08x0.95mm_HandSolder, symbol Device:C_Small
- added D2: D_Small, symbol Device:D_Small
- added D3, D5: LED_Small, LED_SMD:LED_0603_1608Metric_Pad1.05x0.95mm_HandSolder, symbol Device:LED_Small
- added D4: D_Shockley, Diode_THT:D_DO-15_P5.08mm_Vertical_KathodeUp, symbol Device:D_Shockley
- added F1: Polyfuse, Resistor_SMD:R_1812_4532Metric_Pad1.30x3.40mm_HandSolder, symbol Device:Polyfuse
- added FID1: kicad, Symbol:KiCad-Logo2_5mm_SilkScreen, symbol Mechanical:Fiducial
- added FID2: FAN 3d, Z_mycustom_footprint_lib:FAN 80x80x25 12V, symbol Mechanical:Fiducial
- added FID3: Fiducial, Fiducial:Fiducial_0.5mm_Mask1.5mm, symbol Mechanical:Fiducial
- added FID4: trash, Symbol:WEEE-Logo_4.2x6mm_SilkScreen, symbol Mechanical:Fiducial
- added IC1: MCP73834T-FCI_UN, SOP50P490X110-10N, symbol SamacSys_Parts:MCP73834T-FCI_UN
- added J10: HOLE, Connector_PinSocket_2.54mm:PinSocket_1x01_P2.54mm_Vertical, symbol Connector_Generic:Conn_01x01
- added J7, J9: Conn_01x03, Connector_PinHeader_2.54mm:PinHeader_1x03_P2.54mm_Vertical, symbol Connector_Generic:Conn_01x03
- added J8: Out, TerminalBlock:TerminalBlock_Altech_AK300-2_P5.00mm, symbol Connector_Generic:Conn_01x02
- added L2: 1.5u, Inductor_SMD:L_Wuerth_MAPI-3012, symbol Device:L
- added Q2, Q?: Q_NMOS_DGS, symbol Device:Q_NMOS_DGS
- added Q?: Q_PMOS_DGS, symbol Device:Q_PMOS_DGS
- added R2, R21, R22, R24: 10k, symbol Device:R_Small
- added R23, R25, R28: 1Meg, Resistor_SMD:R_0603_1608Metric_Pad0.98x0.95mm_HandSolder, symbol Device:R_Small
- added R26: DNP, Resistor_SMD:R_0603_1608Metric_Pad0.98x0.95mm_HandSolder, symbol Device:R_Small
- added R27: 600, symbol Device:R_Small
- added R29: 180k, Resistor_SMD:R_0603_1608Metric_Pad0.98x0.95mm_HandSolder, symbol Device:R_Small
- added R30, R32: 470, Resistor_SMD:R_0603_1608Metric_Pad0.98x0.95mm_HandSolder, symbol Device:R_Small
- added R31, R33: 10k, Resistor_SMD:R_0603_1608Metric_Pad0.98x0.95mm_HandSolder, symbol Device:R_Small
- added R34, R35: 10k, Resistor_SMD:R_0603_1608Metric_Pad0.98x0.95mm_HandSolder, symbol Device:R
- added R36, R37, R38: 100k, symbol Device:R_Small
- added RV1: R_Potentiometer, symbol Device:R_Potentiometer
- added SW2: RotaryEncoder_Switch, Z_mycustom_footprint_lib:PEC12R4230FS0024, symbol My_custom_lib:RotaryEncoder_Switch
- added SW3: SW_SPDT, Z_mycustom_footprint_lib:SPDT switch 2mm, symbol Switch:SW_SPDT
- added TH1: 68K@25C~5%, Resistor_THT:R_Axial_DIN0204_L3.6mm_D1.6mm_P2.54mm_Vertical, symbol Device:Thermistor_NTC
- added U10: APX810S05, Package_TO_SOT_SMD:SOT-23, symbol My_custom_lib:APX810S05
- added U11: LM2902, symbol Amplifier_Operational:LM2902
- added U7: TPS63020DSJR, Z_mycustom_footprint_lib:TPS63020, symbol My_custom_lib:TPS63020DSJR
- added U9: DMG9933USD-13, Package_SO:SOIC-8_3.9x4.9mm_P1.27mm, symbol My_custom_lib:DMG9933USD-13
- FB1: value FerriteBead_Small -> Ferrite; footprint (none) -> Resistor_SMD:R_0402_1005Metric_Pad0.72x0.64mm_HandSolder
- HS1: value Heatsink_Pad_2Pin -> Heatsink
- J2: value Conn_01x03 -> SWD
- J3: value Screw_Terminal_01x02 -> INPUT
- J4: value Conn_01x02 -> probe
- SW1: footprint (none) -> Z_mycustom_footprint_lib:SPDT switch 2mm
- gave numbers to parts that had none: 10
Connections:
- net +12V: now also U6.4 (V+), C10.1, J7.3 (Pin_3), RV1.1
- net +3.3VA: now also FB1.2, C14.1, R27.2, TH1.1
- net +3V3: now also FB1.1, U5.51 (VCC), C15.1, C16.1, C22.1, Q?.3 (S), R25.1, R26.1, R28.1, SW2.S1, U11.4 (V+), U7.4 (VOUT), U7.5 (VOUT); no longer C6.1, U8.5 (Vin)
- net +5V: now also C20.1, D3.2 (A), D4.2 (A), D5.2 (A), F1.1, IC1.1 (VDD_1), IC1.2 (VDD_2), R35.2, U9.4 (G); no longer FB1.1, U2.5 (VCC)
- net +BATT: now also C21.1, IC1.10 (VBAT_2), IC1.9 (VBAT_1), U10.3 (Vcc), U9.1 (S)
- net ADC_IN1: now also U11.6 (-), U11.7
- net ADC_IN3: now also U11.13 (-), U11.14
- net ADC_IN8: now also U11.1, U11.2 (-)
- net ADC_REF: now also U3.1 (K), C18.2, R27.1
- net GND: now also U3.2 (A), U5.52 (VSS), C13.2, C14.2, C15.2, C16.2, C17.2, C18.1, C19.2, C20.2, C21.2, C22.2, C?.2, D2.1 (K), IC1.5 (VSS), J7.1 (Pin_1), J8.1 (Pin_1), Q2.3 (S), Q?.3 (S), R2.1, R22.1, R23.2, R24.2, R29.2, R31.1, R33.2, R34.1, R35.1, R38.2, RV1.3, SW2.C, SW2.MH (MH2), SW3.3 (C), U10.2 (GND), U11.11 (V-), U7.2 (GND)
- net PWM_SIGNAL3: now also Q?.2 (G), Q?.2 (G)
- net VBUS: now also U2.5 (VCC), F1.2; no longer FB1.2
- net -VDC: now reaches U6.11 (V-)
- net -VDC: now also C10.2, C11.2, C?.1, D2.2 (A), J10.1 (Pin_1), R23.1
- net at U6.1: now also J8.2 (Pin_2), R21.2; no longer U6.2 (-)
- net at U6.3 (+): now also J7.2 (Pin_2), RV1.2
- net at R3.2: now also C13.1, U11.3 (+)
- net at U4.25 (PA15): now also Q2.2 (G), R38.1
- net ENCODER_A: now reaches U4.26 (PB3)
- net ENCODER_A: now also SW2.A
- net ENCODER_B: now reaches U4.27 (PB4)
- net ENCODER_B: now also SW2.B
- net SW_OUT: now reaches U4.28 (PB5)
- net SW_OUT: now also R2.2, SW2.S2
- new net: C11.1, Q?.1 (D), Q?.1 (D)
- new net: IC1.8 (THERM), R31.2
- new net: J9.1 (Pin_1), R21.1
- new net: D5.1 (K), R32.1
- new net: R24.1, TH1.2, U11.12 (+)
- new net: J9.3 (Pin_3), R22.2
- new net: C19.1, SW3.1 (A), U7.1 (VINA), U7.13 (PS/SYNC)
- new net: J9.2 (Pin_2), U6.2 (-)
- new net: IC1.3 (STAT1), R30.2
- new net: IC1.4 (STAT2), R32.2
- new net: L2.2, U7.6 (L2), U7.7 (L2)
- new net: L2.1, U7.8 (L1), U7.9 (L1)
- new net: R36.2, R37.1, U11.5 (+)
- new net: Q2.1 (D), R37.2
- new net: D3.1 (K), R30.1
- new net +VDC: C17.1, C6.1, D4.1 (K), R36.1, U7.10 (VIN), U7.11 (VIN), U8.5 (Vin), U9.3 (S)
- new net Drains: U9.5 (D), U9.6 (D), U9.7 (D), U9.8 (D)
- new net EN_3V3: SW3.2 (B), U7.12 (EN)
- new net FB_3V3: R25.2, R26.2, R29.1, U7.3 (FB)
- new net PG_3V3: R28.2, U7.14 (PG)
- new net Set_charge_current: IC1.6 (PROG), R33.1
- new net TE: IC1.7 (~{PG(}TE))
- new net batt_protection: R34.2, U10.1 (RESET), U9.2 (G)
Other:
- note added: "0.5v FB pin"
- note added: "12V RAIL"
- note added: "3V-3V3"
- note added: "3v3"
- note added: "BATT TO USB POWER AUTO SHITCHING WITH REVERSE POWER PROTECTION"
- note added: "BATT TO USB POWER AUTO SHITCHING WITH REVERSE POWER PROTECTION AND PROTECTED CHARGEING CCCV"
- note added: "ENCODER"
- note added: "LCD"
- note added: "MCU"
- note added: "MOUNTING HOLES FIDUCIALS AND OTHER"
- note added: "PROGRAMABLE LOAD FILTERS AND POWER ELEMENTS"
- note added: "SMALL ADJUSTABLE REFERECE"
- note added: "TE uses 1.8V logic active high activates a timer"
- note added: "USB"
- note added: "VOLTAGE DIVIDER"
- note added: "active when Vbat is under 3.08V active high"
- note added: "https://eu.mouser.com/c/semiconductors/discrete-semiconductors/transistors/mosfet/?channel%20mode=Enhancement&mounting%20style=Through%20Hole&number%20of%20channels=1%20Channel&package%20%2F%20case=TO-92-3&technology=Si&transistor%20polarity=N-Channel&instock=y&sort=pricing"
- note added: "https://eu.mouser.com/c/semiconductors/discrete-semiconductors/transistors/mosfet/?channel%20mode=Enhancement&mounting%20style=Through%20Hole&number%20of%20channels=1%20Channel&package%20%2F%20case=TO-92-3&technology=Si&transistor%20polarity=P-Channel&instock=y&sort=pricing"
- note added: "timer enable"
- moved on the sheet: C1, C2, C3, C4, C5, C6, C7, C8, C9, D1, FB1, H1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

Commit message: n
Parts:
- removed FID2: FAN 3d, Z_mycustom_footprint_lib:FAN 80x80x25 12V, symbol Mechanical:Fiducial
- added C23: 100n, symbol Device:C_Small
- added C24, C25, C26: 47n, symbol Device:C_Small
- added C?: 100n, Capacitor_SMD:C_0603_1608Metric_Pad1.08x0.95mm_HandSolder, symbol Device:C_Small
- added C?: 22u, Capacitor_SMD:C_0805_2012Metric_Pad1.18x1.45mm_HandSolder, symbol Device:C_Small
- added J11: Screw_Terminal_01x03, symbol Connector:Screw_Terminal_01x03
- added J12: LOAD, TerminalBlock:TerminalBlock_Altech_AK300-2_P5.00mm, symbol Connector:Screw_Terminal_01x02
- added Q5: Q_PMOS_DGS, Package_TO_SOT_THT:TO-247-3_Vertical, symbol Device:Q_PMOS_DGS
- added R39, R40, R43, R44, R52: 10k, symbol Device:R_Small
- added R41: 1R, Resistor_THT:R_Axial_Power_L50.0mm_W9.0mm_P55.88mm, symbol Device:R_Small
- added R42, R50, R51: 20k, symbol Device:R_Small
- added R45, R46, R47, R48: 1k, symbol Device:R_Small
- added R49: 100, symbol Device:R_Small
- added U12: LM324A, symbol Amplifier_Operational:LM324A
- added U?: ESP32-S3-WROOM-1, Espressif:ESP32-S3-WROOM-1, symbol Espressif:ESP32-S3-WROOM-1
- HS1: footprint Heatsink:Heatsink_Fischer_SK104-STCB_35x13mm__2xDrill3.5mm_ScrewM3 -> Z_mycustom_footprint_lib:heatsink1
- Q1: footprint Package_TO_SOT_THT:TO-220-3_Vertical -> Package_TO_SOT_THT:TO-247-3_Vertical
- gave numbers to parts that had none: 3
Connections:
- net +12V: now also C23.1, U12.4 (V+)
- net +3V3: now also C?.1, C?.1, U?.2 (3V3)
- net -VDC: now also C23.2, U12.11 (V-)
- net D+: now also U?.14 (GPIO20/U1CTS/ADC2_CH9/CLK_OUT1/USB_D+)
- net D-: now also U?.13 (GPIO19/U1RTS/ADC2_CH8/CLK_OUT2/USB_D-)
- net GND: now also C24.2, C25.2, C26.2, C?.2, C?.2, J11.1 (Pin_1), J12.2 (Pin_2), R40.2, R51.1, R52.1, U?.1 (GND), U?.40 (GND), U?.41 (GND)
- new net: R47.1, U12.1, U12.2 (-)
- new net: C25.1, R47.2, U12.5 (+)
- new net: R39.1, R40.1, U12.12 (+)
- new net: C24.1, R46.2, U12.3 (+)
- new net: C26.1, R45.1, R48.2, U12.10 (+)
- new net: R49.1, U12.8
- new net: R42.1, R51.2, U12.9 (-)
- new net: R48.1, R50.2, U12.7
- new net: Q5.2 (G), R49.2
- new net: J11.2 (Pin_2), R39.2, R41.1, R42.2
- new net: Q5.1 (D), R41.2, R43.1, R45.2
- new net: R43.2, R44.1, U12.13 (-)
- new net: R50.1, R52.2, U12.6 (-)
- new net: J12.1 (Pin_1), Q5.3 (S)
- new net ADC_INx: R44.2, U12.14
- new net BOOT: U?.27 (GPIO0/BOOT)
- new net EN: U?.3 (EN)
- new net GPIO_01: U?.39 (GPIO1/TOUCH1/ADC1_CH0)
- new net GPIO_02: U?.38 (GPIO2/TOUCH2/ADC1_CH1)
- new net GPIO_03: U?.15 (GPIO3/TOUCH3/ADC1_CH2)
- new net GPIO_04: U?.4 (GPIO4/TOUCH4/ADC1_CH3)
- new net GPIO_05: U?.5 (GPIO5/TOUCH5/ADC1_CH4)
- new net GPIO_06: U?.6 (GPIO6/TOUCH6/ADC1_CH5)
- new net GPIO_07: U?.7 (GPIO7/TOUCH7/ADC1_CH6)
- new net GPIO_08: U?.12 (GPIO8/TOUCH8/ADC1_CH7/SUBSPICS1)
- new net GPIO_09: U?.17 (GPIO9/TOUCH9/ADC1_CH8/FSPIHD/SUBSPIHD)
- new net GPIO_10: U?.18 (GPIO10/TOUCH10/ADC1_CH9/FSPICS0/FSPIIO4/SUBSPICS0)
- new net GPIO_11: U?.19 (GPIO11/TOUCH11/ADC2_CH0/FSPID/FSPIIO5/SUBSPID)
- new net GPIO_12: U?.20 (GPIO12/TOUCH12/ADC2_CH1/FSPICLK/FSPIIO6/SUBSPICLK)
- new net GPIO_13: U?.21 (GPIO13/TOUCH13/ADC2_CH2/FSPIQ/FSPIIO7/SUBSPIQ)
- new net GPIO_14: U?.22 (GPIO14/TOUCH14/ADC2_CH3/FSPIWP/FSPIDQS/SUBSPIWP)
- new net GPIO_15: U?.8 (GPIO15/U0RTS/ADC2_CH4/XTAL_32K_P)
- new net GPIO_16: U?.9 (GPIO16/U0CTS/ADC2_CH5/XTAL_32K_NH5)
- new net GPIO_17: U?.10 (GPIO17/U1TXD/ADC2_CH6)
- new net GPIO_18: U?.11 (GPIO18/U1RXD/ADC2_CH7/CLK_OUT3)
- new net GPIO_21: U?.23 (GPIO21)
- new net GPIO_35: U?.28 (SPIIO6/GPIO35/FSPID/SUBSPID)
- new net GPIO_36: U?.29 (SPIIO7/GPIO36/FSPICLK/SUBSPICLK)
- new net GPIO_37: U?.30 (SPIDQS/GPIO37/FSPIQ/SUBSPIQ)
- new net GPIO_38: U?.31 (GPIO38/FSPIWP/SUBSPIWP)
- new net GPIO_39: U?.32 (MTCK/GPIO39/CLK_OUT3/SUBSPICS1)
- new net GPIO_40: U?.33 (MTDO/GPIO40/CLK_OUT2)
- new net GPIO_41: U?.34 (MTDI/GPIO41/CLK_OUT1)
- new net GPIO_42: U?.35 (MTMS/GPIO42)
- new net GPIO_45: U?.26 (GPIO45)
- new net GPIO_46: U?.16 (GPIO46)
- new net GPIO_47: U?.24 (GPIO47/SPICLK_P/SUBSPICLK_P_DIFF)
- new net GPIO_48: U?.25 (GPIO48/SPICLK_N/SUBSPICLK_N_DIFF)
- new net PWM_SIGNALx: R46.1
- new net UART0_RX: U?.37 (U0TXD/GPIO43/CLK_OUT1)
- new net UART0_TX: U?.36 (U0RXD/GPIO44/CLK_OUT2)
- no-connect marks 7 -> 12
Other:
- note added: "Danger free pins:"
- note added: "ESP32-S3 has four strapping pins: • GPIO0 / BOOT • GPIO45 • GPIO46 • GPIO3 GPIO0, GPIO45 and GPIO46 are connected to the chip's internal weak pull-up/pull-down during the chip reset. GPIO3 is floating by default"
- note added: "Free safe pins:"
- note added: "Internal Pull-up/down 45k Max IC typical current: source 40mA sink 28mA EN pin TTL: 0.75*Vcc+ HIGH 0.25*Vcc- LOW"
- moved on the sheet: C1, C10, C11, C12, C13, C14, C15, C16, C17, C18, C19, C2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

Commit message: g
Parts:
- R36, R37: value 100k -> 10k
Connections:
- net ADC_IN1: now also R36.2, R37.1; no longer U11.6 (-), U11.7
- net Cell_measurements_FET: now reaches Q2.2 (G), R38.1
- net Cell_measurements_FET: no longer U4.25 (PA15)
- now unconnected: U11.5 (+)
Other:
- moved on the sheet: C18, Q2, R27, R36, R37, R38, U11B, U3

Commit message: g
Parts:
- removed C10, C18, C22, C23: 100n, symbol Device:C_Small
- removed C11, C12: 47u, Capacitor_THT:CP_Radial_D6.3mm_P2.50mm, symbol Device:C_Small
- removed C13, C24, C25, C26, C7, C8, C9: 47n, symbol Device:C_Small
- removed C15, C17, C?: 22u, Capacitor_SMD:C_0805_2012Metric_Pad1.18x1.45mm_HandSolder, symbol Device:C_Small
- removed C19, C?: 100n, Capacitor_SMD:C_0603_1608Metric_Pad1.08x0.95mm_HandSolder, symbol Device:C_Small
- removed C20: 1u, Capacitor_SMD:C_0603_1608Metric_Pad1.08x0.95mm_HandSolder, symbol Device:C_Small
- removed C21: 4.7u, Capacitor_SMD:C_0603_1608Metric_Pad1.08x0.95mm_HandSolder, symbol Device:C_Small
- removed C6: 4u7, symbol Device:C_Small
- removed R10, R2, R20, R21, R22, R24, R3, R36, R37, R39, R40, R43, R44, R52, R9: 10k, symbol Device:R_Small
- removed R14, R15, R16, R45, R46, R47, R48: 1k, symbol Device:R_Small
- removed R18, R42, R50, R51: 20k, symbol Device:R_Small
- removed R23, R25, R28: 1Meg, Resistor_SMD:R_0603_1608Metric_Pad0.98x0.95mm_HandSolder, symbol Device:R_Small
- removed R27: 600, symbol Device:R_Small
- removed R31, R33: 10k, Resistor_SMD:R_0603_1608Metric_Pad0.98x0.95mm_HandSolder, symbol Device:R_Small
- removed R32: 470, Resistor_SMD:R_0603_1608Metric_Pad0.98x0.95mm_HandSolder, symbol Device:R_Small
- removed R34, R35: 10k, Resistor_SMD:R_0603_1608Metric_Pad0.98x0.95mm_HandSolder, symbol Device:R
- added C? (x8): 47n, Capacitor_SMD:C_0603_1608Metric, symbol Device:C_Small
- added C? (x7): 100n, Capacitor_SMD:C_0603_1608Metric, symbol Device:C_Small
- added C? (x6): 10u, Capacitor_SMD:C_0603_1608Metric, symbol Device:C_Small
- added C? (x6): 22u, Capacitor_SMD:C_0805_2012Metric, symbol Device:C_Small
- added R? (x9): 1k, Resistor_SMD:R_0603_1608Metric, symbol Device:R_Small
- added R? (x20): 10k, Resistor_SMD:R_0603_1608Metric, symbol Device:R_Small
- added R? (x4): 1Meg, Resistor_SMD:R_0603_1608Metric, symbol Device:R_Small
- added R? (x5): 20k, Resistor_SMD:R_0603_1608Metric, symbol Device:R_Small
- added R?: 470, Resistor_SMD:R_0603_1608Metric, symbol Device:R_Small
- C16: footprint Capacitor_SMD:C_0805_2012Metric_Pad1.18x1.45mm_HandSolder -> Capacitor_SMD:C_0805_2012Metric; LCSC (none) -> C45783
- R30: footprint Resistor_SMD:R_0603_1608Metric_Pad0.98x0.95mm_HandSolder -> Resistor_SMD:R_0603_1608Metric; LCSC (none) -> C23179
Connections:
- net +12V: now also C?.1, C?.1
- net +3.3VA: now also R?.2
- net +3V3: now also C?.1, C?.1, C?.1, C?.1, C?.1, R?.2, R?.2
- net +5V: now also C?.1, R?.2
- net +BATT: now also C?.2
- net +VDC: now also C?.2, C?.2, R?.2
- net -VDC: now also C?.1, C?.1, C?.2, C?.2, C?.2, C?.2, R?.2
- net ADC_IN1: now also R?.1, R?.2
- net ADC_INx: now also R?.1
- net ADC_REF: now also C?.1, R?.1
- net FB_3V3: now also R?.1
- net GND: now also C?.1, C?.1, C?.1, C?.2, C?.2, C?.2, C?.2, C?.2, C?.2, C?.2, C?.2, C?.2, C?.2, C?.2, C?.2, C?.2, C?.2, C?.2, C?.2, C?.2, R?.1, R?.1, R?.1, R?.1, R?.1, R?.1, R?.1, R?.1, R?.1, R?.1, R?.1, R?.1, R?.2
- net LOAD: now also R?.2
- net LOAD_VOLTAGE: now also R?.1
- net PG_3V3: now also R?.1
- net PWM_SIGNAL1: now also R?.1
- net PWM_SIGNALx: now also R?.1
- net SW_OUT: now also R?.2
- net Set_charge_current: now also R?.2
- net batt_protection: now also R?.2
- net at U11.3 (+): now also C?.1, R?.2
- net at Q3.1 (D), Q4.1 (D): now also C?.1, C?.1
- net at U6.12 (+): now also C?.1, R?.2
- net at U6.9 (-): now also R?.1, R?.2
- net at U6.8: now also R?.1, R?.2
- net at U12.1, U12.2 (-): now also R?.1
- net at U12.5 (+): now also C?.1, R?.2
- net at U6.13 (-), U6.14: now also R?.1
- net at U6.10 (+): now also C?.1, R?.2
- net at IC1.8 (THERM): now also R?.2
- net at U12.12 (+): now also R?.1, R?.2
- net at J9.1 (Pin_1): now also R?.1
- net at J8.2 (Pin_2), U6.1: now also R?.2
- net at D5.1 (K): now also R?.2
- net at U12.3 (+): now also C?.1, R?.2
- net at TH1.2, U11.12 (+): now also R?.2
- net at U6.5 (+): now also C?.1, R?.2
- net at J5.8 (Pin_8): now also R?.1
- net at J9.3 (Pin_3): now also R?.2
- net at SW3.1 (A), U7.1 (VINA), U7.13 (PS/SYNC): now also C?.1
- net at U12.10 (+): now also C?.1, R?.1, R?.2
- net at U12.9 (-): now also R?.1, R?.2
- net at U12.7: now also R?.1, R?.2
- net at J4.1 (Pin_1), Q1.3 (S), R6.1: now also R?.1
- net at IC1.4 (STAT2): now also R?.1
- net at J11.2 (Pin_2), R41.1: now also R?.2, R?.2
- net at Q5.1 (D), R41.2: now also R?.1, R?.2
- net at Q2.1 (D): now also R?.1
- net at U12.13 (-): now also R?.2, R?.2
- net at U12.6 (-): now also R?.1, R?.2
Other:
- moved on the sheet: C16, D2, Q3, Q4, R38, U11B, U11E, U12E, U6E
