File: Small_load_V1/Small_load_V1.kicad_sch (KiCad schematic)
At the start: 144 parts, among them IC1 MCP73834T-FCI_UN, J1 USB_B, J10 HOLE, J11 Screw_Terminal_01x03, J12 LOAD, J2 SWD, J3 INPUT, J4 probe, J5 Conn_02x04_Odd_Even, J6 Fan, J7 Conn_01x03, J8 Out, J9 Conn_01x03, Q1 IRFZ24NPBF, Q2 Q_NMOS_DGS, Q3 Q_PMOS_DGS, Q4 Q_NMOS_DGS, Q5 Q_PMOS_DGS, SW1 SW_SPDT, SW2 RotaryEncoder_Switch, SW3 SW_SPDT, U1 1043, U10 APX810S05, U11 LM2902, U12 LM324A, U2 D1213A-02SM, U3 LM4040DBZ-2.0, U4 STM32L010K4T6, U5 1602_LCD_I2C, U6 LM324A, U7 TPS63020DSJR, U8 AP3012KTR-G1, U9 DMG9933USD-13

Commit message: f
Parts:
- removed C1: 1u+, symbol Device:C_Small
- removed C3: 100n, symbol Device:C_Small
- removed C? (x2): 100n, Capacitor_SMD:C_0603_1608Metric, symbol Device:C_Small
- removed C? (x4): 22u, Capacitor_SMD:C_0805_2012Metric, symbol Device:C_Small
- removed C? (x2): 10u, Capacitor_SMD:C_0603_1608Metric, symbol Device:C_Small
- removed C?: 47n, Capacitor_SMD:C_0603_1608Metric, symbol Device:C_Small
- removed D4: D_Shockley, Diode_THT:D_DO-15_P5.08mm_Vertical_KathodeUp, symbol Device:D_Shockley
- removed FB1: Ferrite, Resistor_SMD:R_0402_1005Metric_Pad0.72x0.64mm_HandSolder, symbol Device:FerriteBead_Small
- removed J11: Screw_Terminal_01x03, symbol Connector:Screw_Terminal_01x03
- removed J2: SWD, Connector_PinHeader_2.54mm:PinHeader_1x03_P2.54mm_Vertical, symbol Connector_Generic:Conn_01x03
- removed J6: Fan, symbol Connector_Generic:Conn_01x02
- removed J7, J9: Conn_01x03, Connector_PinHeader_2.54mm:PinHeader_1x03_P2.54mm_Vertical, symbol Connector_Generic:Conn_01x03
- removed J8: Out, TerminalBlock:TerminalBlock_Altech_AK300-2_P5.00mm, symbol Connector_Generic:Conn_01x02
- removed L1: 10uH, symbol Device:L
- removed Q3: Q_PMOS_DGS, symbol Device:Q_PMOS_DGS
- removed Q4: Q_NMOS_DGS, symbol Device:Q_NMOS_DGS
- removed R1: 10k, symbol Device:R_Small
- removed R11: 47k, symbol Device:R_Small
- removed R12, R19: 100k, symbol Device:R_Small
- removed R13: 5k1, symbol Device:R_Small
- removed R17, R49: 100, symbol Device:R_Small
- removed R41, R6, R7: 1R, Resistor_THT:R_Axial_Power_L50.0mm_W9.0mm_P55.88mm, symbol Device:R_Small
- removed R? (x2): 1Meg, Resistor_SMD:R_0603_1608Metric, symbol Device:R_Small
- removed R?: 20k, Resistor_SMD:R_0603_1608Metric, symbol Device:R_Small
- removed R? (x3): 10k, Resistor_SMD:R_0603_1608Metric, symbol Device:R_Small
- removed R?: 1k, Resistor_SMD:R_0603_1608Metric, symbol Device:R_Small
- removed RV1: R_Potentiometer, symbol Device:R_Potentiometer
- removed SW1: SW_SPDT, Z_mycustom_footprint_lib:SPDT switch 2mm, symbol Switch:SW_SPDT
- removed TP1: TestPoint, TestPoint:TestPoint_Pad_D2.0mm, symbol Connector:TestPoint
- removed U11: LM2902, symbol Amplifier_Operational:LM2902
- removed U12, U6: LM324A, symbol Amplifier_Operational:LM324A
- removed U4: STM32L010K4T6, Package_QFP:LQFP-32_7x7mm_P0.8mm, symbol MCU_ST_STM32L0:STM32L011K4Tx
- removed U8: AP3012KTR-G1, Package_TO_SOT_SMD:SOT-23-5_HandSoldering, symbol My_custom_lib:AP3012KTR-G1
- added C1, C3: 100n, Capacitor_SMD:C_0603_1608Metric, symbol Device:C
- added C11, C7: 10u, Capacitor_SMD:C_0603_1608Metric, symbol Device:C_Small
- added C12: 47n, Capacitor_SMD:C_0603_1608Metric, symbol Device:C_Small
- added C15, C6: 100n, Capacitor_SMD:C_0603_1608Metric, symbol Device:C_Small
- added D4, D6, D7: B5819W_SL, Diode_SMD:D_SOD-123, symbol Device:D_Small
- added J2: Fan, symbol Connector_Generic:Conn_01x02
- added J3: Input, TerminalBlock:TerminalBlock_Altech_AK300-2_P5.00mm, symbol Connector:Screw_Terminal_01x02
- added L3: 10uH, symbol Device:L
- added R1: 1k, Resistor_SMD:R_0603_1608Metric, symbol Device:R
- added R17, R21: 100k, Resistor_SMD:R_0603_1608Metric, symbol Device:R
- added R2, R63: DNP, Resistor_SMD:R_0603_1608Metric_Pad0.98x0.95mm_HandSolder, symbol Device:R_Small
- added R27, R55: 100, Resistor_SMD:R_0603_1608Metric, symbol Device:R_Small
- added R3, R36, R37, R9: 10k, Resistor_SMD:R_0603_1608Metric, symbol Device:R
- added R30, R64, R65, R68, R71, R77: 100k, Resistor_SMD:R_0603_1608Metric, symbol Device:R_Small
- added R47, R59, R60, R61, R62, R70, R72, R73, R74, R75, R76: 100m, Resistor_SMD:R_0805_2012Metric, symbol Device:R_Small
- added R66, R67: 1k, Resistor_SMD:R_0603_1608Metric, symbol Device:R_Small
- added SW1, SW4: SW_SPST, SamacSys_Parts:PTS526SK15SMTR2LFS, symbol Switch:SW_SPST
- added U1: LM358, Package_SO:SOIC-8_3.9x4.9mm_P1.27mm, symbol Amplifier_Operational:LM358
- added U14: LM324, Package_SO:SOIC-14_3.9x8.7mm_P1.27mm, symbol Amplifier_Operational:LM324
- added U7, U8: LM324, symbol Amplifier_Operational:LM324
- added U9: TPS61040DBV, Package_TO_SOT_SMD:SOT-23-5, symbol Regulator_Switching:TPS61040DBV
- C14: value 100n -> 47n; footprint (none) -> Capacitor_SMD:C_0603_1608Metric; LCSC (none) -> C1622
- C2, C4: value 100n -> 10u; footprint (none) -> Capacitor_SMD:C_0603_1608Metric; LCSC (none) -> C96446
- C5: value 4u7 -> 10u; footprint (none) -> Capacitor_SMD:C_0603_1608Metric; LCSC (none) -> C96446
- D1, D2: value D_Small -> B5819W_SL; footprint (none) -> Diode_SMD:D_SOD-123; LCSC (none) -> C8598
- J4: value probe -> Precision_output; footprint Connector_PinSocket_2.54mm:PinSocket_1x02_P2.54mm_Vertical -> Connector_PinHeader_2.54mm:PinHeader_1x02_P2.54mm_Vertical; now in the parts list
- gave numbers to parts that had none: 51
- renumbered C16 to C10, FID3 to FID2, FID4 to FID3, J5 to J7, J3 to J8, J10 to J9, Q1 to Q3, Q2 to Q4, R4 to R10, R5 to R11, R30 to R12, R8 to R14, R26 to R6, R29 to R8, SW3 to SW2, SW2 to SW3, U1 to U11, U5 to U12, U3 to U13, U7 to U4, U9 to U6
Connections:
- net +12V: now also C15.1, D7.1 (K), J2.2 (Pin_2), R63.1, U14.4 (V+), U7.4 (V+), U8.4 (V+); no longer C5.1, D1.1 (K)
- net +3.3VA: no longer C14.1, R26.2
- net +3V3: now also R26.2, R3.2, R9.2; no longer C2.1
- net +5V: now also D1.2 (A), D4.2 (A)
- net +VDC: now also D1.1 (K), C1.1, C11.2, D4.1 (K), L3.1, U1.8 (V+), U9.4 (EN), U9.5 (VIN)
- net -VDC: now also C4.1, C5.1, R21.1, U7.11 (V-); no longer C22.2
- net BOOT: now also C6.1, R3.1, SW4.2 (B)
- net EN: now also C7.2, R9.1, SW1.2 (B)
- net GND: now also C22.2, J4.1 (Pin_1), C1.2, C11.1, C12.2, C15.2, C3.2, C6.2, C7.1, D6.1 (K), J2.1 (Pin_1), J3.1 (Pin_1), R17.2, R21.2, R30.1, R37.1, R47.2, R59.2, R60.2, R61.2, R62.2, R64.1, R71.2, SW1.1 (A), SW4.1 (A), U1.4 (V-), U14.11 (V-), U8.11 (V-), U9.2 (GND); no longer C2.2, D2.1 (K)
- net at C28.1, R35.2: now also U8.12 (+)
- net at C24.1, R23.2: now also U7.3 (+)
- net at C32.1, R52.2: now also U14.5 (+)
- net at C34.1, R51.1, R54.2: now also U14.10 (+)
- net at R34.2, TH1.2: now also U7.12 (+)
- net at R29.1, R32.2: now also U7.6 (-)
- net at R25.1, R29.2: now also U7.7
- net at C26.1, R25.2: now also U8.3 (+)
- net at C33.1, R53.2: now also U14.12 (+)
- net at R48.1, R57.2: now also U14.9 (-)
- net at Q3.1 (G): now also R27.1
- net at Q3.3 (S), R35.1: now also R47.1, R59.1, R60.1, R61.1, R62.1; no longer J4.1 (Pin_1)
- net at Q5.2 (G): now also R55.1
- net at R45.2, R48.2: now also J3.2 (Pin_2), R72.1, R73.1, R74.1, R75.1, R76.1
- net at R54.1, R56.2: now also U14.14
- net at Q5.1 (D), R49.1, R51.2: now also R72.2, R73.2, R74.2, R75.2, R76.2
- net at R53.1: now also U14.6 (-), U14.7
- net at C25.1, R24.2: now also U7.5 (+)
- net at R56.1, R58.2: now also U14.13 (-)
- net at R24.1: now also U7.1, U7.2 (-)
- net at R45.1, R46.2: now also U7.10 (+)
- net at R49.2, R50.2: now also U7.9 (-)
- net at J4.2 (Pin_2): now also R70.2, U8.10 (+)
- net ADC_IN1 renamed ADC_Batery
- net ADC_INx renamed ADC_Source_current
- net ADC_Source_current: now also U7.8
- net PWM_SIGNAL1 renamed PWM_Signal_Sink
- net PWM_SIGNALx renamed PWM_Signal_Source
- new net: R65.1, R70.1, U8.7
- new net: R65.2, R68.1, U8.6 (-)
- new net: C2.1, R17.1, U1.6 (-), U1.7
- new net: C2.2, D2.1 (K), D6.2 (A)
- new net: R71.1, R77.2, U8.5 (+)
- new net: C3.1, R1.1, R2.2, U1.3 (+)
- new net: R77.1, U8.8, U8.9 (-)
- new net: R63.2, R64.2, U9.3 (FB)
- new net: D7.2 (A), L3.2, U9.1 (SW)
- new net: R27.2, R30.2, U8.1, U8.2 (-)
- new net: R55.2, U14.8
- new net: C14.1, R67.2, R68.2
- new net: C12.1, R66.2, U14.3 (+)
- new net: R67.1, U14.1, U14.2 (-)
- new net ADC_Sink_current: U8.13 (-), U8.14
- new net ADC_heatsink: U7.13 (-), U7.14
- new net PWM_precise_source: R66.1
- new net PWM_pump: R1.2, R2.1, R36.2, U1.1, U1.5 (+)
- new net fb__pump: R36.1, R37.2, U1.2 (-)
- no-connect marks 12 -> 11
Other:
- note added: "+"
- note added: "Iout= Vin*A/shunt A=Rin/Rother"
- note removed: "12.77V"
- note removed: "12V RAIL"
- note removed: "LOW ==> OFF HIGH==> ON"
- note removed: "SMALL ADJUSTABLE REFERECE"
- note removed: "USB"
- note removed: "https://eu.mouser.com/c/semiconductors/discrete-semiconductors/transistors/mosfet/?channel%20mode=Enhancement&mounting%20style=Through%20Hole&number%20of%20channels=1%20Channel&package%20%2F%20case=TO-92-3&technology=Si&transistor%20polarity=N-Channel&instock=y&sort=pricing"
- note removed: "https://eu.mouser.com/c/semiconductors/discrete-semiconductors/transistors/mosfet/?channel%20mode=Enhancement&mounting%20style=Through%20Hole&number%20of%20channels=1%20Channel&package%20%2F%20case=TO-92-3&technology=Si&transistor%20polarity=P-Channel&instock=y&sort=pricing"
- moved on the sheet: C10, C13, C19, C21, C22, C23, C27, C8, C9, D3, D5, F1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

Commit message: g
Parts:
- removed C1, C3: 100n, Capacitor_SMD:C_0603_1608Metric, symbol Device:C
- removed C10, C8, C9: 22u, Capacitor_SMD:C_0805_2012Metric, symbol Device:C_Small
- removed C11, C16, C17, C2, C4: 10u, Capacitor_SMD:C_0603_1608Metric, symbol Device:C_Small
- removed C12, C24, C25, C26, C28, C32, C33, C34: 47n, Capacitor_SMD:C_0603_1608Metric, symbol Device:C_Small
- removed C18, C22, C27: 100n, Capacitor_SMD:C_0603_1608Metric, symbol Device:C_Small
- removed D2, D6, D7: B5819W_SL, Diode_SMD:D_SOD-123, symbol Device:D_Small
- removed J12: LOAD, TerminalBlock:TerminalBlock_Altech_AK300-2_P5.00mm, symbol Connector:Screw_Terminal_01x02
- removed J2: Fan, symbol Connector_Generic:Conn_01x02
- removed J4: Precision_output, Connector_PinHeader_2.54mm:PinHeader_1x02_P2.54mm_Vertical, symbol Connector_Generic:Conn_01x02
- removed J7: Conn_02x04_Odd_Even, Connector_PinHeader_2.54mm:PinHeader_2x04_P2.54mm_Vertical, symbol Connector_Generic:Conn_02x04_Odd_Even
- removed L2: 1.5u, Inductor_SMD:L_Wuerth_MAPI-3012, symbol Device:L
- removed L3: 10uH, symbol Device:L
- removed Q4: Q_NMOS_DGS, symbol Device:Q_NMOS_DGS
- removed Q5: Q_PMOS_DGS, Package_TO_SOT_THT:TO-247-3_Vertical, symbol Device:Q_PMOS_DGS
- removed R1: 1k, Resistor_SMD:R_0603_1608Metric, symbol Device:R
- removed R10: 65k, symbol Device:R_Small
- removed R14: X, Resistor_THT:R_Axial_DIN0207_L6.3mm_D2.5mm_P10.16mm_Horizontal, symbol Device:R_Small
- removed R15, R22, R28, R32, R33, R34, R35, R45, R46, R49, R50, R58: 10k, Resistor_SMD:R_0603_1608Metric, symbol Device:R_Small
- removed R17, R21: 100k, Resistor_SMD:R_0603_1608Metric, symbol Device:R
- removed R2, R63: DNP, Resistor_SMD:R_0603_1608Metric_Pad0.98x0.95mm_HandSolder, symbol Device:R_Small
- removed R23, R24, R25, R26, R51, R52, R53, R54, R66, R67: 1k, Resistor_SMD:R_0603_1608Metric, symbol Device:R_Small
- removed R29, R48, R56, R57: 20k, Resistor_SMD:R_0603_1608Metric, symbol Device:R_Small
- removed R30, R64, R65, R68, R71, R77: 100k, Resistor_SMD:R_0603_1608Metric, symbol Device:R_Small
- removed R36, R37: 10k, Resistor_SMD:R_0603_1608Metric, symbol Device:R
- removed R38: 100k, symbol Device:R_Small
- removed R55: 100, Resistor_SMD:R_0603_1608Metric, symbol Device:R_Small
- removed R59, R60, R61, R62, R70, R72, R73, R74, R75, R76: 100m, Resistor_SMD:R_0805_2012Metric, symbol Device:R_Small
- removed SW2: SW_SPDT, Z_mycustom_footprint_lib:SPDT switch 2mm, symbol Switch:SW_SPDT
- removed TH1: 68K@25C~5%, Resistor_THT:R_Axial_DIN0204_L3.6mm_D1.6mm_P2.54mm_Vertical, symbol Device:Thermistor_NTC
- removed U1: LM358, Package_SO:SOIC-8_3.9x4.9mm_P1.27mm, symbol Amplifier_Operational:LM358
- removed U11: 1043, 1043, symbol SamacSys_Parts:1043
- removed U13: LM4040DBZ-2.0, Package_TO_SOT_SMD:SOT-23, symbol Reference_Voltage:LM4040DBZ-2.0
- removed U14: LM324, Package_SO:SOIC-14_3.9x8.7mm_P1.27mm, symbol Amplifier_Operational:LM324
- removed U2: D1213A-02SM, Package_TO_SOT_SMD:SOT-23-5_HandSoldering, symbol My_custom_lib:D1213A-02SM
- removed U4: TPS63020DSJR, Z_mycustom_footprint_lib:TPS63020, symbol My_custom_lib:TPS63020DSJR
- removed U5: ESP32-S3-WROOM-1, Espressif:ESP32-S3-WROOM-1, symbol Espressif:ESP32-S3-WROOM-1
- removed U7, U8: LM324, symbol Amplifier_Operational:LM324
- removed U9: TPS61040DBV, Package_TO_SOT_SMD:SOT-23-5, symbol Regulator_Switching:TPS61040DBV
- added C3: 100p, Capacitor_SMD:C_0603_1608Metric, symbol Device:C_Small
- added C33 (x2), C57: 1u, Capacitor_SMD:C_0402_1005Metric, symbol Device:C_Small
- added D6, D7: green, LED_SMD:LED_0805_2012Metric, symbol Device:LED_Small
- added FID1 (x2): Polarity, Symbol:Polarity_Center_Positive_6mm_SilkScreen, symbol Mechanical:Fiducial
- added J11: Li ION cell own power, Z_mycustom_footprint_lib:MYOUNG MY-18650-01, symbol Connector_Generic:Conn_01x02
- added J14 (x2): Jack-DC, Connector_BarrelJack:BarrelJack_Wuerth_6941xx301002, symbol Connector:Jack-DC
- added JP1: Jumper_2_Bridged, Jumper:SolderJumper-2_P1.3mm_Bridged_RoundedPad1.0x1.5mm, symbol Jumper:Jumper_2_Bridged
- added Q1: IRF9540N, Package_TO_SOT_THT:TO-220-3_Vertical, symbol Transistor_FET:IRF9540N
- added R1: 15-16k, Resistor_SMD:R_0603_1608Metric, symbol Device:R_Small
- added R13 (x2): 2k, Resistor_SMD:R_0402_1005Metric, symbol Device:R_Small
- added R13: 470, Resistor_SMD:R_0402_1005Metric, symbol Device:R_Small
- added R40, R41 (x2): 1k, Resistor_SMD:R_0805_2012Metric, symbol Device:R
- added U11: AD5337, Package_SO:MSOP-8_3x3mm_P0.65mm, symbol My_custom_lib:AD5337
- added U2, U7, U8: AD8001AR, Package_SO:SOIC-8_3.9x4.9mm_P1.27mm, symbol Amplifier_Operational:AD8001AR
- added U3: ESP32-S3-WROOM-1, Espressif:ESP32-S3-WROOM-1, symbol Espressif:ESP32-S3-WROOM-1
- added U4: MCP3208, Package_SO:SOIC-16_3.9x9.9mm_P1.27mm, symbol Analog_ADC:MCP3208
- added U4: SRV05-4, Package_TO_SOT_SMD:SOT-23-6, symbol Power_Protection:SRV05-4
- added U9: CJ431, Package_TO_SOT_SMD:SOT-23, symbol My_custom_lib:CJ431
- C13: value 100n -> 1u; footprint Capacitor_SMD:C_0603_1608Metric -> Capacitor_SMD:C_0402_1005Metric; LCSC C14663 -> C52923
- C14: value 47n -> 10u; LCSC C1622 -> C96446
- C15: value 100n -> 10u; LCSC C14663 -> C96446
- C5: value 10u -> 100p; LCSC C96446 -> C14663
- C7: value 10u -> 100n; LCSC C19702 -> C14663
- R11: value 65k -> 50m; footprint (none) -> Resistor_THT:R_Axial_DIN0516_L15.5mm_D5.0mm_P20.32mm_Horizontal
- R47: value 100m -> 50m; footprint Resistor_SMD:R_0805_2012Metric -> Resistor_THT:R_Axial_DIN0516_L15.5mm_D5.0mm_P20.32mm_Horizontal; LCSC C25334 -> (none)
- R5: value 1Meg -> 100; LCSC C22935 -> C22775
- R6: value DNP -> 10k; footprint Resistor_SMD:R_0603_1608Metric_Pad0.98x0.95mm_HandSolder -> Resistor_SMD:R_0603_1608Metric; LCSC (none) -> C25804
- R7: value 1Meg -> 10k; LCSC C22935 -> C25804
- R8: value 180k -> 10k; footprint Resistor_SMD:R_0603_1608Metric_Pad0.98x0.95mm_HandSolder -> Resistor_SMD:R_0603_1608Metric; LCSC (none) -> C25804
Connections:
- net +12V: no longer C15.1
- net +3V3: now also C13.2, C14.1, C15.1, C33.2, C33.2, D7.2 (A), U11.1 (VDD), U3.2 (3V3), U4.16 (Vdd); no longer R5.2, R6.1, R7.2
- net +5V: now also D6.2 (A)
- net +BATT: now also J11.1 (Pin_1)
- net +VDC: now also R13.1, R13.2
- net -VDC: no longer C5.1
- net BOOT: now also U3.27 (GPIO0/BOOT)
- net D+: now also U3.14 (GPIO20/U1CTS/ADC2_CH9/CLK_OUT1/USB_D+), U4.1 (IO1)
- net D-: now also U3.13 (GPIO19/U1RTS/ADC2_CH8/CLK_OUT2/USB_D-), U4.6 (IO4)
- net EN: now also C7.1, U3.3 (EN); no longer C7.2
- net GND: now also C13.1, C7.2, R8.1, C33.1, C33.1, C57.1, J11.2 (Pin_2), J14.2, J14.2, JP1.1 (A), R1.1, R13.2, U11.5 (GND), U11.8 (A0), U3.1 (GND), U3.40 (GND), U3.41 (GND), U4.14 (AGND), U4.2 (VN), U4.9 (DGND), U9.3 (A); no longer C13.2, C5.2, C7.1, R8.2
- net LOAD: now also J14.1; no longer R11.2
- net UART0_RX: now also U3.37 (U0TXD/GPIO43/CLK_OUT1)
- net UART0_TX: now also U3.36 (U0RXD/GPIO44/CLK_OUT2)
- net VBUS: now also U4.5 (VP)
- net at J3.2 (Pin_2): now also R11.1, R7.2, J14.1, U8.3 (+)
- net at Q3.3 (S), R47.1: now also R41.2
- net at R27.2: now also C3.1, U2.6
- removed net FB_3V3: R5.1, R6.2, R8.1
- net PG_3V3: no longer names the net of R7.1
- net PG_3V3: now also R13.1
- new net: D6.1 (K), R40.1
- new net: C5.2, R6.1, R8.2, U7.3 (+)
- new net: D7.1 (K), R41.1
- new net: Q1.1 (G), R5.1
- new net: R5.2, U7.6
- new net: C5.1, Q1.2 (D), R6.2
- new net: Q1.3 (S), R11.2, U8.2 (-)
- new net: JP1.2 (B), R40.2, R41.2
- new net: C3.2, R1.2, R41.1, U2.2 (-)
- new net DAC1: U11.2 (Vout_A), U2.3 (+)
- new net DAC2: U11.3 (Vout_B), U7.2 (-)
- new net REF_2v5: C57.2, R13.1, R13.2, U11.4 (REF), U4.15 (Vref), U9.1 (REF), U9.2 (K)
- new net SCL: U11.7 (SCL)
- new net SDA: U11.6 (SDA)
- no-connect marks 11 -> 9
Other:
- note added: "50m 2W"
- note added: "DAC adress: 000110[A0] 0x0C or 0x0D"
- note added: "Turn on output = 0V So buck Vout is 5.5V !! Or 4.45V IF DAC is tristate"
- note added: "USB+ESC TVS + Indicator LEDs"
- note removed: "+"
- note removed: "0.5v FB pin"
- note removed: "3V-3V3"
- note removed: "3v3"
- note removed: "Free safe pins:"
- note removed: "Iout= Vin*A/shunt A=Rin/Rother"
- note removed: "Max voltage: 2V"
- note removed: "THT custom"
- note removed: "VOLTAGE DIVIDER"
- note removed: "from left to right:"
- note removed: "max voltage 55V"
- note removed: "normal 12-15V line"
- moved on the sheet: C19, C21, C23, C6, D1, D3, D4, D5, F1, FID1, FID2, FID3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

Commit message: f
Parts:
- removed C33, C57: 1u, Capacitor_SMD:C_0402_1005Metric, symbol Device:C_Small
- removed R13: 2k, Resistor_SMD:R_0402_1005Metric, symbol Device:R_Small
- removed R13: 470, Resistor_SMD:R_0402_1005Metric, symbol Device:R_Small
- removed U4: MCP3208, Package_SO:SOIC-16_3.9x9.9mm_P1.27mm, symbol Analog_ADC:MCP3208
- removed U9: CJ431, Package_TO_SOT_SMD:SOT-23, symbol My_custom_lib:CJ431
Other:
- added sheet Cell_balancer (Cell_balancer.kicad_sch)
- moved on the sheet: C19, C21, C23, C3, C33, C5, D1, D3, D4, D5, D6, D7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

Commit message: g
Parts:
- removed C19, C23: 10u, Capacitor_SMD:C_0603_1608Metric, symbol Device:C_Small
- removed D1, D4: B5819W_SL, Diode_SMD:D_SOD-123, symbol Device:D_Small
- removed D3, D5: LED_Small, LED_SMD:LED_0603_1608Metric_Pad1.05x0.95mm_HandSolder, symbol Device:LED_Small
- removed IC1: MCP73834T-FCI_UN, SOP50P490X110-10N, symbol SamacSys_Parts:MCP73834T-FCI_UN
- removed J3: Input, TerminalBlock:TerminalBlock_Altech_AK300-2_P5.00mm, symbol Connector:Screw_Terminal_01x02
- removed J9: HOLE, Connector_PinSocket_2.54mm:PinSocket_1x01_P2.54mm_Vertical, symbol Connector_Generic:Conn_01x01
- removed Q1: IRF9540N, Package_TO_SOT_THT:TO-220-3_Vertical, symbol Transistor_FET:IRF9540N
- removed R13, R19, R20: 10k, Resistor_SMD:R_0603_1608Metric, symbol Device:R_Small
- removed R13: 2k, Resistor_SMD:R_0402_1005Metric, symbol Device:R_Small
- removed R40, R41 (x2): 1k, Resistor_SMD:R_0805_2012Metric, symbol Device:R
- removed R5: 100, Resistor_SMD:R_0603_1608Metric, symbol Device:R_Small
- removed U10: APX810S05, Package_TO_SOT_SMD:SOT-23, symbol My_custom_lib:APX810S05
- removed U6: DMG9933USD-13, Package_SO:SOIC-8_3.9x4.9mm_P1.27mm, symbol My_custom_lib:DMG9933USD-13
- removed U7, U8: AD8001AR, Package_SO:SOIC-8_3.9x4.9mm_P1.27mm, symbol Amplifier_Operational:AD8001AR
- added C33 (x2), C57: 1u, Capacitor_SMD:C_0402_1005Metric, symbol Device:C_Small
- added C56: 100p, Capacitor_SMD:C_0603_1608Metric, symbol Device:C_Small
- added D4, D5: 1N4007, Diode_THT:D_DO-41_SOD81_P10.16mm_Horizontal, symbol Diode:1N4007
- added J11: Input, TerminalBlock:TerminalBlock_Altech_AK300-2_P5.00mm, symbol Connector:Screw_Terminal_01x02
- added J2: Conn_01x06, symbol Connector_Generic:Conn_01x06
- added Q1, Q2: 2N7002, Package_TO_SOT_SMD:SOT-23, symbol Transistor_FET:2N7002
- added Q10: IRFZ24NPBF, Package_TO_SOT_THT:TO-247-3_Vertical, symbol Device:Q_NMOS_GDS
- added Q5: IRF9540N, Package_TO_SOT_THT:TO-220-3_Vertical, symbol Transistor_FET:IRF9540N
- added Q7: 2N3904, Package_TO_SOT_THT:TO-92_Inline, symbol Transistor_BJT:2N3904
- added R10, R2, R26, R28, R30: 1k, Resistor_SMD:R_0603_1608Metric, symbol Device:R_Small
- added R13: 2k, Resistor_SMD:R_0402_1005Metric, symbol Device:R_Small
- added R13: 1k, Resistor_THT:R_Axial_DIN0309_L9.0mm_D3.2mm_P5.08mm_Vertical, symbol Device:R_Small
- added R13: 470, Resistor_SMD:R_0402_1005Metric, symbol Device:R_Small
- added R14, R17, R24, R29, R32, R46, R48: 10k, Resistor_SMD:R_0603_1608Metric, symbol Device:R_Small
- added R15, R25: 100, Resistor_SMD:R_0603_1608Metric, symbol Device:R_Small
- added R22: 1, Resistor_THT:R_Axial_DIN0516_L15.5mm_D5.0mm_P20.32mm_Horizontal, symbol Device:R_Small
- added R41: 50m, Resistor_THT:R_Axial_DIN0516_L15.5mm_D5.0mm_P20.32mm_Horizontal, symbol Device:R_Small
- added U11: AD5337, Package_SO:MSOP-8_3x3mm_P0.65mm, symbol My_custom_lib:AD5337
- added unit 4 of U11
- added U13, U7, U8: LM324A, Package_SO:SOIC-14_3.9x8.7mm_P1.27mm, symbol Amplifier_Operational:LM324A
- added U4: MCP3208, Package_SO:SOIC-16_3.9x9.9mm_P1.27mm, symbol Analog_ADC:MCP3208
- added U9: AD8001AR, Package_SO:SOIC-8_3.9x4.9mm_P1.27mm, symbol Amplifier_Operational:AD8001AR
- added U9: CJ431, Package_TO_SOT_SMD:SOT-23, symbol My_custom_lib:CJ431
- C5: value 100p -> 100n
- R1: value 15-16k -> 3k; LCSC C25804 -> C4211
- R11: value 50m -> 1k; footprint Resistor_THT:R_Axial_DIN0516_L15.5mm_D5.0mm_P20.32mm_Horizontal -> Resistor_SMD:R_0603_1608Metric; LCSC (none) -> C21190
- R12: value 470 -> 1k; LCSC C23179 -> C21190
- R16: value 470 -> 10k; LCSC C23179 -> C25804
- R6, R8: value 10k -> 1k; LCSC C25804 -> C21190
- R7: value 10k -> 3k; LCSC C25804 -> C4211
- U12: footprint Z_mycustom_footprint_lib:1602 LCD I2C -> Z_mycustom_footprint_lib:1602_LCD_mine; now not fitted; now left out of the parts list
Connections:
- net Set_charge_current is gone; now on net +3V3: R18.2
- net +3V3: now also C33.2, C33.2, Q1.1 (G), Q2.1 (G), R13.1, R13.2, R13.2, R17.2, U11.1 (VDD), U4.16 (Vdd)
- net +5V: now also R16.2, J2.1 (Pin_1), R14.2
- net DAC2: now also U9.3 (+)
- net GND: now also C5.2, R7.1, C33.1, C33.1, C57.1, D4.1 (K), J11.1 (Pin_1), J2.4 (Pin_4), J2.6 (Pin_6), Q7.1 (E), R22.2, R28.2, R46.1, U11.5 (GND), U11.8 (A0), U4.14 (AGND), U4.9 (DGND), U9.3 (A); no longer R18.1, R8.1
- net I2C_CLK: now also R16.1, J2.3 (Pin_3), Q2.3 (D); no longer U12.54 (SCL)
- net I2C_SDA: now also J2.2 (Pin_2), Q1.3 (D), R14.1; no longer U12.53 (SDA)
- net LOAD: now also Q10.2 (D)
- net REF_2v5: now also C5.1, C57.2, R13.1, R13.2, U11.4 (REF), U4.15 (Vref), U9.1 (REF), U9.2 (K)
- net SCL: now also U11.7 (SCL)
- net SDA: now also U11.6 (SDA)
- net at D6.1 (K): now also R8.1
- net at D7.1 (K): now also R10.1
- net at R6.2: now also C3.2, R1.2, U2.2 (-); no longer C5.1
- net at R11.2: now also R48.2, U7.13 (-)
- net at Q3.3 (S), R47.1: now also R6.1
- net at R12.2: now also R46.2, U7.12 (+)
- net at JP1.2 (B): now also R8.2, R10.2
- net LDO_Vcc: now reaches R12.1
- net LDO_Vcc: now also J14.1, J11.2 (Pin_2), R41.1
- new net: R30.1, R32.1, U13.13 (-)
- new net: Q7.2 (B), R24.1
- new net: Q7.3 (C), R25.1, R26.1
- new net: R26.2, U11.14
- new net: J2.5 (Pin_5), R13.1
- new net: R48.1, U7.14, U8.13 (-)
- new net: R25.2, R29.2, U13.12 (+)
- new net: Q5.1 (G), U13.14
- new net: D4.2 (A), D5.1 (K)
- new net: Q5.3 (S), R11.1, R41.2
- new net: C56.2, R2.2, R7.2, U9.2 (-)
- new net: C56.1, R15.2, U9.6
- new net: Q10.3 (S), R2.1, R22.1
- new net: Q10.1 (G), R15.1
- new net: R24.2, U8.14
- new net: D5.2 (A), R30.2
- new net: R28.1, R29.1, U11.13 (-)
- new net DAC3: U11.2 (Vout_A), U8.12 (+)
- new net DAC4: U11.12 (+), U11.3 (Vout_B)
- new net I2C_CLK_3V3: Q2.2 (S), R18.1
- new net I2C_SDA_3V3: Q1.2 (S), R17.1
- new net VLDO_OUT: Q5.2 (D), R32.2
- no-connect marks 9 -> 7
Other:
- removed sheet Cell_balancer
- added sheet buck (buck.kicad_sch)
- note added: "0-2.5V scale 0 0 1v 0.25A 2V 0.5A 0.5*1 = 0.5V => 0.5V/2v => x4 gain"
- note added: "0-2.5V scale 0 0 1v 5A 2V 10A 10*0.05 = 0.5V => 0.5V/2v => x4 gain"
- note added: "1 2W"
- note removed: "BATT TO USB POWER AUTO SHITCHING WITH REVERSE POWER PROTECTION"
- note removed: "BATT TO USB POWER AUTO SHITCHING WITH REVERSE POWER PROTECTION AND PROTECTED CHARGEING CCCV"
- note removed: "TE uses 1.8V logic active high activates a timer"
- note removed: "active when Vbat is under 3.08V active high"
- note removed: "timer enable"
- moved on the sheet: C21, C33, D6, D7, F1, J1, J11, JP1, R31, U11, U4
