File: Small_load_V1/Small_load_V1.kicad_sch (KiCad schematic)
At the start: 89 parts, among them J1 USB_B, J11 Input, J11 Li ION cell own power, J14 Jack-DC, J2 Conn_01x06, J8 INPUT, Q1 2N7002, Q10 IRFZ24NPBF, Q2 2N7002, Q3 IRFZ24NPBF, Q5 IRF9540N, Q7 2N3904, SW1 SW_SPST, SW3 RotaryEncoder_Switch, SW4 SW_SPST, U11 AD5337, U12 1602_LCD_I2C, U13 LM324A, U2 AD8001AR, U3 ESP32-S3-WROOM-1, U4 MCP3208, U4 SRV05-4, U7 LM324A, U8 LM324A, U9 AD8001AR, U9 CJ431

Commit message: g
Parts:
- removed D4, D5: 1N4007, Diode_THT:D_DO-41_SOD81_P10.16mm_Horizontal, symbol Diode:1N4007
- removed J11: Li ION cell own power, Z_mycustom_footprint_lib:MYOUNG MY-18650-01, symbol Connector_Generic:Conn_01x02
- removed Q5: IRF9540N, Package_TO_SOT_THT:TO-220-3_Vertical, symbol Transistor_FET:IRF9540N
- removed Q7: 2N3904, Package_TO_SOT_THT:TO-92_Inline, symbol Transistor_BJT:2N3904
- removed R28, R30: 1k, Resistor_SMD:R_0603_1608Metric, symbol Device:R_Small
- removed R29, R48: 10k, Resistor_SMD:R_0603_1608Metric, symbol Device:R_Small
- removed unit 4 of U11
- removed U13, U7, U8: LM324A, Package_SO:SOIC-14_3.9x8.7mm_P1.27mm, symbol Amplifier_Operational:LM324A
- removed U2, U9: AD8001AR, Package_SO:SOIC-8_3.9x4.9mm_P1.27mm, symbol Amplifier_Operational:AD8001AR
- added C11, C23: 100n, Capacitor_SMD:C_0603_1608Metric, symbol Device:C_Small
- added C22: 100p, Capacitor_SMD:C_0603_1608Metric, symbol Device:C_Small
- added C33: 1u, Capacitor_SMD:C_0402_1005Metric, symbol Device:C_Small
- added C57, C7: 10u, Capacitor_SMD:C_0603_1608Metric, symbol Device:C_Small
- added C63: 4n7, Capacitor_SMD:C_0402_1005Metric, symbol Device:C_Small
- added D1, D2: LED_Small, LED_SMD:LED_0805_2012Metric, symbol Device:LED_Small
- added D4: SS54, Diode_SMD:D_SMA, symbol Device:D_Schottky
- added J7: Input, TerminalBlock:TerminalBlock_Altech_AK300-2_P5.00mm, symbol Connector:Screw_Terminal_01x02
- added Q5: Q_PMOS_DGS, symbol Device:Q_PMOS_DGS
- added Q7: 2N7002, Package_TO_SOT_SMD:SOT-23, symbol Transistor_FET:2N7002
- added R10, R6, R9: 300, Resistor_SMD:R_0603_1608Metric_Pad0.98x0.95mm_HandSolder, symbol Device:R_Small
- added R20: 56, Resistor_SMD:R_0603_1608Metric, symbol Device:R_Small
- added R23, R64: 5R1, Resistor_SMD:R_0402_1005Metric, symbol Device:R_Small
- added R33: 1k, Resistor_SMD:R_0603_1608Metric, symbol Device:R_Small
- added R34, R35, R36, R42, R43, R53, R55: 10k, Resistor_SMD:R_0603_1608Metric, symbol Device:R_Small
- added R44: 2.7M, Resistor_SMD:R_0603_1608Metric, symbol Device:R_Small
- added R51: 330k, Resistor_SMD:R_0603_1608Metric, symbol Device:R_Small
- added R52: 1M, Resistor_SMD:R_0603_1608Metric, symbol Device:R_Small
- added R72: 0R1, Resistor_SMD:R_1206_3216Metric, symbol Device:R_Small
- added U1: CH340C, Package_SO:SOIC-16_3.9x9.9mm_P1.27mm, symbol Interface_USB:CH340C
- added U2, U8: LM324, Package_SO:SOIC-14_3.9x8.7mm_P1.27mm, symbol Amplifier_Operational:LM324
- added U3: AMS1117-3.3, Package_TO_SOT_SMD:SOT-223-3_TabPin2, symbol Regulator_Linear:AMS1117-3.3
- added U7: LT3080xQ, Package_TO_SOT_SMD:TO-263-5_TabPin3, symbol Regulator_Linear:LT3080xQ
- R25: value 100 -> 50m; footprint Resistor_SMD:R_0603_1608Metric -> Resistor_THT:R_Axial_DIN0516_L15.5mm_D5.0mm_P20.32mm_Horizontal; LCSC C22775 -> (none)
- R26: value 1k -> 100; LCSC C21190 -> C22775
- R32: value 10k -> 16k; LCSC C25804 -> (none)
- R41: value 50m -> 10k; footprint Resistor_THT:R_Axial_DIN0516_L15.5mm_D5.0mm_P20.32mm_Horizontal -> Resistor_SMD:R_0603_1608Metric; LCSC (none) -> C25804
Connections:
- net +12V is gone; now on net +5V: C21.1
- net -VDC is gone; now on net GND: C21.2
- net VLDO_OUT is gone; now on an unnamed net: R32.2
- net +3V3: now also R41.2, U11.8 (A0), C33.2, C57.1, D1.2 (A), D2.2 (A), R34.2, R35.2, R36.2, R53.2, U3.2 (VO), U8.5 (VS)
- net +5V: now also C7.1, U1.16 (VCC), U3.3 (VI), U8.4 (V+)
- net D+: now also U1.5 (UD+); no longer U3.14 (GPIO20/U1CTS/ADC2_CH9/CLK_OUT1/USB_D+)
- net D-: now also U1.6 (UD-); no longer U3.13 (GPIO19/U1RTS/ADC2_CH8/CLK_OUT2/USB_D-)
- net DAC1: now also U8.3 (+)
- net DAC2: now also U8.5 (+)
- net DAC3: now also U2.10 (+)
- net DAC4: now also U2.12 (+)
- net GND: now also R11.2, R12.2, C11.2, C23.2, C33.1, C57.2, C7.2, J7.1 (Pin_1), Q7.2 (S), R33.2, R42.1, R43.1, R52.1, R55.1, U1.1 (GND), U2.11 (V-), U2.3 (+), U3.1 (GND), U8.1 (A1), U8.11 (V-), U8.2 (A0), U8.6 (GND); no longer R46.1, U11.8 (A0)
- net LDO_Vcc: now also R46.2, C11.1, C22.1, D4.1 (K), Q5.3 (S), U2.4 (V+); no longer R12.1, R41.1
- net LOAD: now also R44.2
- net SCL: now also R41.1, U8.4 (SCL)
- net SDA: now also R36.1, U8.3 (SDA)
- net UART0_RX: now also R9.1, U1.2 (TXD)
- net UART0_TX: now also R10.1, R6.1
- net at R32.1: now also R33.1, U2.13 (-)
- net at R24.1: now also R11.1, U2.9 (-)
- net at R26.1: now also C22.2, Q5.2 (G); no longer R25.1
- net at R26.2: now also U2.14
- net at Q3.3 (S), R47.1, R6.1: now also U8.12 (+)
- net at C3.1, R27.2: now also U8.1
- net at C3.2, R1.2, R6.2: now also U8.2 (-)
- net at R25.2: now also U7.4 (VCONTROL), U7.5 (IN)
- net at C56.2, R2.2, R7.2: now also U8.6 (-)
- net at C56.1, R15.2: now also U8.7
- net SPI_SS1: now reaches U4.10 (~{CS}/SHDN)
- net SPI_MOSI: now reaches U4.11 (Din)
- net SPI_MISO: now reaches U4.12 (Dout)
- net SPI_clk: now reaches U4.13 (CLK)
- net at R24.2: now also U2.8, U7.2 (SET)
- new net: R12.1, R46.1, U2.5 (+)
- new net: D4.2 (A), R23.1, R72.2, U7.3 (OUT), U7.6 (OUT)
- new net: C23.1, U1.4 (V3)
- new net: C63.2, R64.2, U8.7 (IN-)
- new net: R6.2, U1.3 (RXD)
- new net: Q5.1 (D), R25.1
- new net: D2.1 (K), R10.2
- new net: R44.1, R51.2, R52.2, U8.10 (+)
- new net: C63.1, R23.2, U8.8 (IN+)
- new net: Q7.1 (G), R20.1, R53.1
- new net: D1.1 (K), R9.2
- new net: Q7.3 (D), R51.1
- new net: U2.1, U2.2 (-)
- new net Divider_nmos: R20.2
- new net LDO_Vin: R55.2, U2.6 (-), U2.7
- new net LDO_Vout: J7.2 (Pin_2), R64.1, R72.1
- new net Load_current_main: R42.2, U8.13 (-), U8.14
- new net Load_voltage: R43.2, U8.8, U8.9 (-)
- new net SCL1: R35.1
- new net SDA1: R34.1
- new net ~{DTR}: U1.13 (~{DTR})
- new net ~{RTS}: U1.14 (~{RTS})
- no-connect marks 7 -> 16
Other:
- added sheet CELL_CHARGER (CELL_CHARGER.kicad_sch)
- note added: "1/12"
- note added: "3Meg totalis ok"
- note removed: "18650 cell holder"
- note removed: "Turn on output = 0V So buck Vout is 5.5V !! Or 4.45V IF DAC is tristate"
- moved on the sheet: C21, C33, C5, C57, F1, FID1, J1, J11, J14, J2, Q1, Q2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

Commit message: v
Parts:
- removed C56: 100p, Capacitor_SMD:C_0603_1608Metric, symbol Device:C_Small
- removed F1: Polyfuse, Resistor_SMD:R_1812_4532Metric_Pad1.30x3.40mm_HandSolder, symbol Device:Polyfuse
- removed Q5: Q_PMOS_DGS, symbol Device:Q_PMOS_DGS
- removed R25: 50m, Resistor_THT:R_Axial_DIN0516_L15.5mm_D5.0mm_P20.32mm_Horizontal, symbol Device:R_Small
- removed R35: 10k, Resistor_SMD:R_0603_1608Metric, symbol Device:R_Small
- removed U3: ESP32-S3-WROOM-1, Espressif:ESP32-S3-WROOM-1, symbol Espressif:ESP32-S3-WROOM-1
- removed U4: SRV05-4, Package_TO_SOT_SMD:SOT-23-6, symbol Power_Protection:SRV05-4
- added C13: 1u, Capacitor_SMD:C_0402_1005Metric, symbol Device:C_Small
- added C27: 100u, Capacitor_THT:CP_Radial_D8.0mm_P3.50mm, symbol Device:C_Polarized_Small
- added C34, C45: 100n, Capacitor_SMD:C_0603_1608Metric, symbol Device:C_Small
- added C37: 100p, Capacitor_SMD:C_0402_1005Metric, symbol Device:C_Small
- added C8: 10u@50V, Capacitor_SMD:C_0805_2012Metric, symbol Device:C
- added D8, D9: ZMMxx, Diode_SMD:D_MiniMELF, symbol Diode:ZMMxx
- added J14: USB_C_Receptacle, Z_mycustom_footprint_lib:MC-710, symbol Connector:USB_C_Receptacle
- added J16: Input, TerminalBlock:TerminalBlock_Altech_AK300-2_P5.00mm, symbol Connector:Screw_Terminal_01x02
- added Q5: 2N7002, Package_TO_SOT_SMD:SOT-23, symbol Transistor_FET:2N7002
- added Q8: IRF9530NPBF, Package_TO_SOT_THT:TO-220-3_Vertical, symbol Device:Q_PMOS_GDS
- added R23 (x2): 10, Resistor_SMD:R_0402_1005Metric, symbol Device:R_Small
- added R65, R79, R81, R83, R85: 10k, Resistor_SMD:R_0603_1608Metric, symbol Device:R_Small
- added R72 (x3): 0R1, Resistor_SMD:R_1206_3216Metric, symbol Device:R_Small
- added R82: 1M, Resistor_SMD:R_0603_1608Metric, symbol Device:R_Small
- added R84: 1k, Resistor_SMD:R_0603_1608Metric, symbol Device:R_Small
- added U15: CH224K, Z_mycustom_footprint_lib:CH224K, symbol My_custom_lib:CH224K
- added U19: LM324A, Package_SO:SOIC-14_3.9x8.7mm_P1.27mm, symbol Amplifier_Operational:LM324A
- added U3: ESP32-S3-WROOM-1, PCM_Espressif:ESP32-S3-WROOM-1, symbol PCM_Espressif:ESP32-S3-WROOM-1
- C3: footprint Capacitor_SMD:C_0603_1608Metric -> Capacitor_SMD:C_0402_1005Metric; LCSC C14663 -> C1546
- J2: value Conn_01x06 -> LCD_conn; footprint (none) -> Connector_PinHeader_2.54mm:PinHeader_1x06_P2.54mm_Vertical
- R23, R64: value 5R1 -> 10
- R24, R46: value 10k -> 15k; LCSC C25804 -> C22809
- R32: value 16k -> 15k; LCSC (none) -> C22809
- R51: LCSC (none) -> C23137
- R52: LCSC (none) -> C22935
Connections:
- net I2C_CLK_3V3 is gone; now on net SCL1: Q2.2 (S), R18.1
- net I2C_SDA_3V3 is gone; now on net SDA1: Q1.2 (S), R17.1
- net VBUS is gone; now on net +5V: J1.1 (VBUS)
- net +3V3: now also R79.2, U3.2 (3V3); no longer U11.8 (A0)
- net +5V: now also J2.6 (Pin_6), C45.1, U19.4 (V+); no longer J2.1 (Pin_1)
- net BOOT: now also U3.27 (GPIO0/BOOT)
- net BUCK_EN: now also U3.7 (GPIO7/TOUCH7/ADC1_CH6)
- net D+: now also J14.A6 (D+), J14.B6 (D+), U15.4 (D+), U3.14 (GPIO20/U1CTS/ADC2_CH9/CLK_OUT1/USB_D+); no longer J1.3 (D+), U1.5 (UD+)
- net D-: now also J14.A7 (D-), J14.B7 (D-), U15.5 (D-), U3.13 (GPIO19/U1RTS/ADC2_CH8/CLK_OUT2/USB_D-); no longer J1.2 (D-), U1.6 (UD-)
- net DAC1: now also U8.5 (+); no longer U8.3 (+)
- net DAC2: now also U8.10 (+); no longer U8.5 (+)
- net Divider_nmos: now also U3.22 (GPIO14/TOUCH14/ADC2_CH3/FSPIWP/FSPIDQS/SUBSPIWP)
- net EN: now also U3.3 (EN)
- net ENCODER_A: now also R23.2
- net ENCODER_B: now also R23.2
- net GND: now also J2.1 (Pin_1), J2.3 (Pin_3), C13.1, C27.2, C34.2, C45.2, C8.1, D8.2 (A), J14.A1 (GND), J14.A12 (GND), J14.B1 (GND), J14.B12 (GND), J16.1 (Pin_1), Q5.2 (S), R65.1, R85.1, U15.0 (GND), U19.11 (V-), U3.1 (GND), U3.40 (GND), U3.41 (GND); no longer J2.4 (Pin_4), J2.6 (Pin_6)
- net I2C_CLK: now also J2.4 (Pin_4); no longer J2.3 (Pin_3)
- net I2C_SDA: now also J2.5 (Pin_5); no longer J2.2 (Pin_2)
- net LDO_Vcc: now also Q8.3 (S)
- net LDO_Vin: now also U4.8 (CH7)
- net LDO_Vout: now also C34.1, C8.2, R72.1
- net LOAD: now also C27.1
- net Load_current_main: now also U4.5 (CH4), U8.1, U8.2 (-); no longer U8.13 (-), U8.14
- net Load_voltage: now also U4.6 (CH5), U8.13 (-), U8.14; no longer U8.8, U8.9 (-)
- net SCL: now also U3.17 (GPIO9/TOUCH9/ADC1_CH8/FSPIHD/SUBSPIHD)
- net SCL1: now also U3.10 (GPIO17/U1TXD/ADC2_CH6)
- net SDA: now also U3.12 (GPIO8/TOUCH8/ADC1_CH7/SUBSPICS1)
- net SDA1: now also U3.11 (GPIO18/U1RXD/ADC2_CH7/CLK_OUT3); no longer R34.1
- net SPI_MISO: now also U3.21 (GPIO13/TOUCH13/ADC2_CH2/FSPIQ/FSPIIO7/SUBSPIQ)
- net SPI_MOSI: now also U3.19 (GPIO11/TOUCH11/ADC2_CH0/FSPID/FSPIIO5/SUBSPID)
- net SPI_SS1: now also R34.1, U3.18 (GPIO10/TOUCH10/ADC1_CH9/FSPICS0/FSPIIO4/SUBSPICS0)
- net SPI_clk: now also U3.20 (GPIO12/TOUCH12/ADC2_CH1/FSPICLK/FSPIIO6/SUBSPICLK)
- net SW_OUT: now also U3.32 (MTCK/GPIO39/CLK_OUT3/SUBSPICS1)
- net UART0_RX: now also U3.37 (U0TXD/GPIO43/CLK_OUT1)
- net UART0_TX: now also U3.36 (U0RXD/GPIO44/CLK_OUT2)
- net LT3080_output: now reaches D4.2 (A), R23.1, R72.2, U7.3 (OUT), U7.6 (OUT)
- net LT3080_output: now also R72.2
- net LT3080_input: now reaches R32.2, U7.4 (VCONTROL), U7.5 (IN)
- net LT3080_input: now also R72.1, R72.1
- net at C22.2, R26.1: now also Q8.1 (G)
- net at C3.1, R27.2: now also U8.7; no longer U8.1
- net at C3.2, R1.2, R6.2: now also U8.6 (-); no longer U8.2 (-)
- net at Q3.3 (S), R47.1, R6.1: now also U8.3 (+); no longer U8.12 (+)
- net at R13.1: now also J2.2 (Pin_2); no longer J2.5 (Pin_5)
- net at R44.1, R51.2, R52.2: now also U8.12 (+); no longer U8.10 (+)
- net at Q10.3 (S), R2.1, R22.1: now also U19.12 (+)
- net at R2.2, R7.2: now also U8.9 (-), C37.2; no longer U8.6 (-)
- net Load_current_small: now reaches U4.1 (CH0)
- net Load_current_small: now also R65.2, U19.13 (-), U19.14
- net SMPS_current: now reaches U4.2 (CH1)
- net SMPS_output: now reaches U4.3 (CH2)
- net SMPS_input: now reaches U4.4 (CH3)
- net at R15.2: now also U8.8, C37.1; no longer U8.7
- new net: Q8.2 (D), R72.2, R72.2
- new net: J14.A4 (VBUS), J14.A9 (VBUS), J14.B4 (VBUS), J14.B9 (VBUS), J16.2 (Pin_2), R83.2, R84.1
- new net: C13.2, D9.1 (K), R81.2, R82.2, R84.2, U15.1 (Vdd)
- new net: R82.1, U15.10 (PG)
- new net: R83.1, U15.8 (Vbus)
- new net: D8.1 (K), D9.2 (A)
- new net: R79.1, U11.8 (A0)
- new net: R23.1, U3.34 (MTDI/GPIO41/CLK_OUT1)
- new net: R23.1, U3.35 (MTMS/GPIO42)
- new net CC1: J14.A5 (CC1), U15.6 (CC2)
- new net CC2: J14.B5 (CC2), U15.7 (CC1)
- new net CFG1: Q5.3 (D), R81.1, U15.9 (CFG1)
- new net CFG1_gate: Q5.1 (G), R85.2, U3.4 (GPIO4/TOUCH4/ADC1_CH3)
- new net CFG2: U15.2 (CFG2), U3.5 (GPIO5/TOUCH5/ADC1_CH4)
- new net CFG3: U15.3 (CFG3), U3.6 (GPIO6/TOUCH6/ADC1_CH5)
- new net DD+: J1.3 (D+), U1.5 (UD+)
- new net DD-: J1.2 (D-), U1.6 (UD-)
- new net Driver_High_gate: U3.28 (SPIIO6/GPIO35/FSPID/SUBSPID)
- new net Driver_Low_gate: U3.29 (SPIIO7/GPIO36/FSPICLK/SUBSPICLK)
- no-connect marks 16 -> 24
Other:
- note added: "+-26V max"
- note added: "36V max"
- note added: "40V"
- moved on the sheet: C13, C14, C15, C21, C23, C3, C33, C57, C6, C7, D1, D2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
