File: Small_load_V1/Cell_balancer.kicad_sch (KiCad schematic)
At the start: 56 parts, among them J6 Conn_01x08, Q2 AGM420MC, Q4 AGM420MC, Q5 AGM420MC, Q6 AGM420MC, Q7 AGM420MC, Q8 AGM420MC, Q9 AGM420MC, U4 MCP3208, U9 CJ431

Commit message: g
Parts:
- removed C57: 1u, Capacitor_SMD:C_0402_1005Metric, symbol Device:C_Small
- removed R13: 2k, Resistor_SMD:R_0402_1005Metric, symbol Device:R_Small
- removed R13: 470, Resistor_SMD:R_0402_1005Metric, symbol Device:R_Small
- removed U9: CJ431, Package_TO_SOT_SMD:SOT-23, symbol My_custom_lib:CJ431
