File: Small_load_V1/Small_load_V1.kicad_pcb (KiCad board)
At the start: 2 copper layers, 100 x 100 mm, 12 parts, among them J3 Conn_01x02, Q1 IRFZ24NPBF, U1 D1213A-02SM, U2 STM32L010K4T6, U3 1043

Commit message: f
Parts:
- moved J3 99.5 mm to (102.6, 112.3)
- moved U1 99.5 mm to (107.8, 112.3)
Changed lines of the file:
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@@
     (pad "1" thru_hole circle (at 12.7 0) (size 6 6) (drill 3.5) (layers *.Cu *.Mask)
       (net 1 "GND") (pintype "passive"))
-    (model "${KICAD6_3DMODEL_DIR}/Heatsink.3dshapes/Heatsink_Fischer_SK104-STCB_35x13mm__2xDrill3.5mm_ScrewM3.wrl"
-      (offset (xyz 0 0 0))
-      (scale (xyz 1 1 1))
-      (rotate (xyz 0 0 0))
+    (model "C:/Users/robert_alfred.kecs/Documents/KiCad/my_3D_models/random_from_online/CUI_DEVICES_HSE-B20500-040H-01.step"
+      (offset (xyz 0 0 1))
+      (scale (xyz 1 1 1))
+      (rotate (xyz 180 0 0))
     )
   )
@@
   )
   (footprint "Connector_PinSocket_2.54mm:PinSocket_1x02_P2.54mm_Vertical" (layer "F.Cu")
-    (at 198.6534 86.4108)
+    (at 102.5906 112.3442)
     (descr "Through hole straight socket strip, 1x02, 2.54mm pitch, single row (from Kicad 4.0.7), script generated")
     (tags "Through hole socket strip THT 1x02 2.54mm single row")
@@
   )
   (footprint "Package_TO_SOT_SMD:SOT-23-5_HandSoldering" (layer "F.Cu")
-    (at 203.8334 86.4108)
+    (at 107.7706 112.3442)
     (descr "5-pin SOT23 package")
     (tags "SOT-23-5 hand-soldering")

Commit message: b
Parts:
- added J1: USB_B, Connector_USB:USB_A_CONNFLY_DS1095-WNR0, F.Cu at (63.5, 75.2)
- added J2: Conn_01x03, Connector_PinHeader_2.54mm:PinHeader_1x03_P2.54mm_Vertical, F.Cu at (136.2, 185.1)
- added J3: Screw_Terminal_01x02, TerminalBlock:TerminalBlock_Altech_AK300-2_P5.00mm, F.Cu at (114.0, 58.2)
- added J5: Conn_02x04_Odd_Even, Connector_PinHeader_2.54mm:PinHeader_2x04_P2.54mm_Vertical, F.Cu at (136.2, 172.9)
- added R8: X, Resistor_THT:R_Axial_DIN0207_L6.3mm_D2.5mm_P10.16mm_Horizontal, F.Cu at (95.2, 170.9)
- added TP1: TestPoint, TestPoint:TestPoint_Pad_D2.0mm, F.Cu at (117.4, 170.9)
- added U3: LM4040DBZ-2.0, Package_TO_SOT_SMD:SOT-23, F.Cu at (96.1, 175.2)
- added U5: 1602_LCD_I2C, Z_mycustom_footprint_lib:1602 LCD I2C, F.Cu at (68.8, 98.6)
- added U6: LM324A, Package_SO:SOIC-14_3.9x8.7mm_P1.27mm, F.Cu at (111.2, 174.0)
- moved HS1 74.0 mm to (121.2, 142.0), turned to 180 degrees
- moved Q1 64.8 mm to (123.6, 137.5), turned to 180 degrees
- moved J4 59.4 mm to (129.3, 165.4)
- moved U2 51.3 mm to (68.6, 79.2), turned to -90 degrees
- moved R7 46.9 mm to (142.7, 124.7), turned to 90 degrees
- moved R6 45.7 mm to (132.2, 124.7), turned to 90 degrees
- moved U1 2.88 mm to (67.6, 135.7)
- renumbered J3 to J4, R2 to R6, R4 to R7, U3 to U1, U1 to U2, U2 to U4
Connections:
- Q1 pad 2: Net-(J2-Pad1) -> LOAD
- U2 pad 3: D+ -> D-
- U2 pad 4: D- -> D+
- U4 pad 10: unconnected-(U2-Pad10) -> SPI_SS
- U4 pad 11: unconnected-(U2-Pad11) -> SPI_CLK
- U4 pad 12: unconnected-(U2-Pad12) -> SPI_MOSI
- U4 pad 13: unconnected-(U2-Pad13) -> SPI_MISO
- U4 pad 14: unconnected-(U2-Pad14) -> ADC_IN8
- U4 pad 15: unconnected-(U2-Pad15) -> ADC_REF
- U4 pad 18: unconnected-(U2-Pad18) -> Crystal_Clock_out
- U4 pad 19: unconnected-(U2-Pad19) -> I2C_CLK
- U4 pad 20: unconnected-(U2-Pad20) -> I2C_SDA
- U4 pad 23: unconnected-(U2-Pad23) -> SWD_DIO
- U4 pad 24: unconnected-(U2-Pad24) -> SWD_CLK
- U4 pad 6: unconnected-(U2-Pad6) -> CLOCK_in
- U4 pad 7: unconnected-(U2-Pad7) -> ADC_IN1
- U4 pad 8: unconnected-(U2-Pad8) -> SYS_wakeup3
- U4 pad 9: unconnected-(U2-Pad9) -> ADC_IN3

Commit message: ;
Parts:
- added C11: 1u, Capacitor_SMD:C_0603_1608Metric_Pad1.08x0.95mm_HandSolder, F.Cu at (184.5, 150.6)
- added C12: 100n, Capacitor_SMD:C_0603_1608Metric_Pad1.08x0.95mm_HandSolder, F.Cu at (184.5, 153.1)
- added C15: 22u, Capacitor_SMD:C_0805_2012Metric_Pad1.18x1.45mm_HandSolder, F.Cu at (179.5, 191.0)
- added C16: 22u, Capacitor_SMD:C_0805_2012Metric_Pad1.18x1.45mm_HandSolder, F.Cu at (184.3, 191.0)
- added C17: 22u, Capacitor_SMD:C_0805_2012Metric_Pad1.18x1.45mm_HandSolder, F.Cu at (195.2, 181.2)
- added C19: 100n, Capacitor_SMD:C_0603_1608Metric_Pad1.08x0.95mm_HandSolder, F.Cu at (200.2, 182.1)
- added C20: 1u, Capacitor_SMD:C_0603_1608Metric_Pad1.08x0.95mm_HandSolder, F.Cu at (204.1, 179.6)
- added C21: 4.7u, Capacitor_SMD:C_0603_1608Metric_Pad1.08x0.95mm_HandSolder, F.Cu at (200.2, 184.6)
- added D3: LED_Small, LED_SMD:LED_0603_1608Metric_Pad1.05x0.95mm_HandSolder, F.Cu at (191.5, 185.9)
- added D4: D_Shockley, Diode_THT:D_DO-15_P5.08mm_Vertical_KathodeUp, F.Cu at (179.0, 175.8)
- added D5: LED_Small, LED_SMD:LED_0603_1608Metric_Pad1.05x0.95mm_HandSolder, F.Cu at (201.4, 174.5)
- added F1: Polyfuse, Resistor_SMD:R_1812_4532Metric_Pad1.30x3.40mm_HandSolder, F.Cu at (189.1, 182.2)
- added FB1: Ferrite, Resistor_SMD:R_0402_1005Metric_Pad0.72x0.64mm_HandSolder, F.Cu at (209.6, 174.2)
- added FID1: kicad, Symbol:KiCad-Logo2_5mm_SilkScreen, F.Cu at (207.2, 122.2)
- added FID2: FAN 3d, Z_mycustom_footprint_lib:FAN 80x80x25 12V, F.Cu at (240.9, 95.1)
- added FID3: Fiducial, Fiducial:Fiducial_0.5mm_Mask1.5mm, F.Cu at (201.9, 127.2)
- added FID4: trash, Symbol:WEEE-Logo_4.2x6mm_SilkScreen, F.Cu at (228.7, 122.2)
- added IC1: MCP73834T-FCI_UN, SamacSys_Parts:SOP50P490X110-10N, F.Cu at (180.7, 187.1)
- added J10: HOLE, Connector_PinSocket_2.54mm:PinSocket_1x01_P2.54mm_Vertical, F.Cu at (66.3, 178.8)
- added J7: Conn_01x03, Connector_PinHeader_2.54mm:PinHeader_1x03_P2.54mm_Vertical, F.Cu at (95.8, 185.7)
- added J8: Out, TerminalBlock:TerminalBlock_Altech_AK300-2_P5.00mm, F.Cu at (116.6, 57.4)
- added J9: Conn_01x03, Connector_PinHeader_2.54mm:PinHeader_1x03_P2.54mm_Vertical, F.Cu at (83.5, 199.7)
- added L2: 1.5u, Inductor_SMD:L_Wuerth_MAPI-3012, F.Cu at (196.7, 175.7)
- added R23: 47k, Resistor_SMD:R_0603_1608Metric_Pad0.98x0.95mm_HandSolder, F.Cu at (188.8, 150.6)
- added R25: 1Meg, Resistor_SMD:R_0603_1608Metric_Pad0.98x0.95mm_HandSolder, F.Cu at (210.1, 177.0)
- added R26: DNP, Resistor_SMD:R_0603_1608Metric_Pad0.98x0.95mm_HandSolder, F.Cu at (195.9, 184.0)
- added R28: 1Meg, Resistor_SMD:R_0603_1608Metric_Pad0.98x0.95mm_HandSolder, F.Cu at (205.8, 174.5)
- added R29: 180k, Resistor_SMD:R_0603_1608Metric_Pad0.98x0.95mm_HandSolder, F.Cu at (199.8, 179.6)
- added R30: 470, Resistor_SMD:R_0603_1608Metric_Pad0.98x0.95mm_HandSolder, F.Cu at (195.9, 186.5)
- added R31: 10k, Resistor_SMD:R_0603_1608Metric_Pad0.98x0.95mm_HandSolder, F.Cu at (201.4, 177.0)
- added R32: 470, Resistor_SMD:R_0603_1608Metric_Pad0.98x0.95mm_HandSolder, F.Cu at (205.8, 177.0)
- added R33: 10k, Resistor_SMD:R_0603_1608Metric_Pad0.98x0.95mm_HandSolder, F.Cu at (191.5, 188.5)
- added R34: 10k, Resistor_SMD:R_0603_1608Metric_Pad0.98x0.95mm_HandSolder, F.Cu at (193.2, 191.0)
- added R35: 10k, Resistor_SMD:R_0603_1608Metric_Pad0.98x0.95mm_HandSolder, F.Cu at (188.8, 191.0)
- added SW1: SW_SPDT, Z_mycustom_footprint_lib:SPDT switch 2mm, F.Cu at (287.6, 74.1)
- added SW2: RotaryEncoder_Switch, Z_mycustom_footprint_lib:PEC12R4230FS0024, F.Cu at (97.3, 54.4)
- added SW3: SW_SPDT, Z_mycustom_footprint_lib:SPDT switch 2mm, F.Cu at (220.0, 121.3)
- added TH1: 68K@25C~5%, Resistor_THT:R_Axial_DIN0204_L3.6mm_D1.6mm_P2.54mm_Vertical, F.Cu at (188.4, 92.9)
- added U10: APX810S05, Package_TO_SOT_SMD:SOT-23, F.Cu at (186.8, 187.0)
- added U11: LM2902, Package_SO:SOIC-14_3.9x8.7mm_P1.27mm, F.Cu at (285.7, 81.8)
- added U7: TPS63020DSJR, Z_mycustom_footprint_lib:TPS63020, F.Cu at (190.2, 176.3)
- added U8: AP3012KTR-G1, Package_TO_SOT_SMD:SOT-23-5_HandSoldering, F.Cu at (101.0, 185.7)
- added U9: DMG9933USD-13, Package_SO:SOIC-8_3.9x4.9mm_P1.27mm, F.Cu at (181.3, 181.6)
- HS1: value Heatsink_Pad_2Pin -> Heatsink
- J2: value Conn_01x03 -> SWD
- J3: value Screw_Terminal_01x02 -> INPUT
- J4: value Conn_01x02 -> probe
- R6: moved to B.Cu
- moved J4 36.8 mm to (141.2, 130.6), turned to 90 degrees
- moved U4 20.6 mm to (80.3, 83.1)
- moved J3 16.0 mm to (130.1, 57.4)
- moved R6 8.87 mm to (141.0, 125.7)
- moved R7 1.33 mm to (144.0, 125.2)
Connections:
- J5 pad 1: Net-(J5-Pad1) -> LOAD_VOLTAGE
- J5 pad 3: Net-(J5-Pad1) -> LOAD_VOLTAGE
- J5 pad 5: Net-(J5-Pad1) -> LOAD_VOLTAGE
- J5 pad 7: Net-(J5-Pad1) -> LOAD_VOLTAGE
- Q1 pad 1: unconnected-(Q1-Pad1) -> Net-(Q1-Pad1)
- U2 pad 5: +5V -> VBUS
- U3 pad 1: unconnected-(U3-Pad1) -> ADC_REF
- U3 pad 2: unconnected-(U3-Pad2) -> GND
- U4 pad 25: unconnected-(U4-Pad25) -> Net-(U4-Pad25)
- U4 pad 26: unconnected-(U4-Pad26) -> /ENCODER_A
- U4 pad 27: unconnected-(U4-Pad27) -> /ENCODER_B
- U4 pad 28: unconnected-(U4-Pad28) -> /SW_OUT
- U6 pad 1: unconnected-(U6-Pad1) -> Net-(J8-Pad2)
- U6 pad 10: unconnected-(U6-Pad10) -> Net-(C8-Pad1)
- U6 pad 11: unconnected-(U6-Pad11) -> GND
- U6 pad 12: Net-(J5-Pad1) -> Net-(C7-Pad1)
- U6 pad 13: LOAD_VOLTAGE -> Net-(R15-Pad1)
- U6 pad 14: LOAD_VOLTAGE -> Net-(R15-Pad1)
- U6 pad 2: unconnected-(U6-Pad2) -> Net-(J9-Pad2)
- U6 pad 3: unconnected-(U6-Pad3) -> Net-(J7-Pad2)
- U6 pad 4: unconnected-(U6-Pad4) -> +12V
- U6 pad 5: unconnected-(U6-Pad5) -> Net-(C9-Pad1)
- U6 pad 6: unconnected-(U6-Pad6) -> Net-(R17-Pad1)
- U6 pad 7: unconnected-(U6-Pad7) -> Net-(R17-Pad1)
- U6 pad 8: unconnected-(U6-Pad8) -> Net-(R16-Pad1)
- U6 pad 9: unconnected-(U6-Pad9) -> Net-(R18-Pad1)

Commit message: n
Parts:
- removed FID2: FAN 3d, Z_mycustom_footprint_lib:FAN 80x80x25 12V
- added J12: LOAD, TerminalBlock:TerminalBlock_Altech_AK300-2_P5.00mm, F.Cu at (275.5, 144.5)
- added Q5: Q_PMOS_DGS, Package_TO_SOT_THT:TO-247-3_Vertical, F.Cu at (117.7, 123.1)
- added R41: 1R, Resistor_THT:R_Axial_Power_L50.0mm_W9.0mm_P55.88mm, F.Cu at (214.3, 142.8)
- C11: value 1u -> 47u; footprint Capacitor_SMD:C_0603_1608Metric_Pad1.08x0.95mm_HandSolder -> Capacitor_THT:CP_Radial_D6.3mm_P2.50mm
- C12: value 100n -> 47u; footprint Capacitor_SMD:C_0603_1608Metric_Pad1.08x0.95mm_HandSolder -> Capacitor_THT:CP_Radial_D6.3mm_P2.50mm
- HS1: footprint Heatsink:Heatsink_Fischer_SK104-STCB_35x13mm__2xDrill3.5mm_ScrewM3 -> Z_mycustom_footprint_lib:heatsink1
- Q1: footprint Package_TO_SOT_THT:TO-220-3_Vertical -> Package_TO_SOT_THT:TO-247-3_Vertical
- R23: value 47k -> 1Meg
- moved R6 199.6 mm to (332.0, 67.4)
- moved R7 199.6 mm to (334.9, 67.0)
- moved J3 87.7 mm to (214.4, 33.5)
- moved J8 87.7 mm to (200.9, 33.5)
- moved J4 72.3 mm to (145.2, 202.8)
- moved Q1 39.0 mm to (117.8, 99.0), turned to -90 degrees
- moved C11 10.8 mm to (195.1, 148.5)
- moved C12 6.34 mm to (178.4, 155.0)
- moved HS1 5.63 mm to (123.7, 147.0), turned to 90 degrees
- moved TP1 4.38 mm to (121.7, 171.9)
Connections:
- net PWM_SIGNAL3 renamed Net-(C11-Pad1)
- C11 pad 2: /LCD_BIAS -> -VDC
- C12 pad 1: /LCD_BIAS -> -VDC
- J10 pad 1: /LCD_BIAS -> -VDC
- R23 pad 1: /LCD_BIAS -> -VDC
- U6 pad 11: GND -> -VDC

Commit message: f
Parts:
- removed C20: 1u, Capacitor_SMD:C_0603_1608Metric_Pad1.08x0.95mm_HandSolder
- removed FB1: Ferrite, Resistor_SMD:R_0402_1005Metric_Pad0.72x0.64mm_HandSolder
- removed FID4: trash, Symbol:WEEE-Logo_4.2x6mm_SilkScreen
- removed J10: HOLE, Connector_PinSocket_2.54mm:PinSocket_1x01_P2.54mm_Vertical
- removed J2: SWD, Connector_PinHeader_2.54mm:PinHeader_1x03_P2.54mm_Vertical
- removed J5: Conn_02x04_Odd_Even, Connector_PinHeader_2.54mm:PinHeader_2x04_P2.54mm_Vertical
- removed Q1: IRFZ24NPBF, Package_TO_SOT_THT:TO-247-3_Vertical
- removed TP1: TestPoint, TestPoint:TestPoint_Pad_D2.0mm
- removed U3: LM4040DBZ-2.0, Package_TO_SOT_SMD:SOT-23
- added C1: 100n, Capacitor_SMD:C_0603_1608Metric, F.Cu at (265.6, 94.0)
- added C10: 22u, Capacitor_SMD:C_0805_2012Metric, F.Cu at (293.5, 54.1)
- added C13: 100n, Capacitor_SMD:C_0603_1608Metric, F.Cu at (296.0, 66.9)
- added C14: 47n, Capacitor_SMD:C_0603_1608Metric, F.Cu at (286.6, 75.8)
- added C18: 100n, Capacitor_SMD:C_0603_1608Metric, F.Cu at (234.1, 131.1)
- added C2: 10u, Capacitor_SMD:C_0603_1608Metric, F.Cu at (279.2, 81.4)
- added C22: 100n, Capacitor_SMD:C_0603_1608Metric, F.Cu at (278.5, 76.4)
- added C23: 10u, Capacitor_SMD:C_0603_1608Metric, F.Cu at (261.6, 110.7)
- added C24: 47n, Capacitor_SMD:C_0603_1608Metric, F.Cu at (226.1, 128.5)
- added C25: 47n, Capacitor_SMD:C_0603_1608Metric, F.Cu at (297.3, 56.9)
- added C26: 47n, Capacitor_SMD:C_0603_1608Metric, F.Cu at (309.3, 56.4)
- added C27: 100n, Capacitor_SMD:C_0603_1608Metric, F.Cu at (230.1, 128.5)
- added C28: 47n, Capacitor_SMD:C_0603_1608Metric, F.Cu at (261.6, 108.2)
- added C29: 10u, Capacitor_SMD:C_0603_1608Metric, F.Cu at (271.2, 81.2)
- added C3: 100n, Capacitor_SMD:C_0603_1608Metric, F.Cu at (268.6, 86.4)
- added C30: 100n, Capacitor_SMD:C_0603_1608Metric, F.Cu at (288.0, 68.5)
- added C31: 47n, Capacitor_SMD:C_0603_1608Metric, F.Cu at (240.7, 115.9)
- added C32: 47n, Capacitor_SMD:C_0603_1608Metric, F.Cu at (268.5, 88.9)
- added C33: 47n, Capacitor_SMD:C_0603_1608Metric, F.Cu at (309.7, 53.9)
- added C34: 47n, Capacitor_SMD:C_0603_1608Metric, F.Cu at (237.9, 123.4)
- added C4: 10u, Capacitor_SMD:C_0603_1608Metric, F.Cu at (297.6, 59.4)
- added C5: 10u, Capacitor_SMD:C_0603_1608Metric, F.Cu at (275.2, 81.4)
- added C6: 100n, Capacitor_SMD:C_0603_1608Metric, F.Cu at (228.3, 99.3)
- added C7: 10u, Capacitor_SMD:C_0603_1608Metric, F.Cu at (234.5, 125.9)
- added C8: 22u, Capacitor_SMD:C_0805_2012Metric, F.Cu at (225.7, 120.8)
- added C9: 22u, Capacitor_SMD:C_0805_2012Metric, F.Cu at (285.4, 61.5)
- added D1: B5819W_SL, Diode_SMD:D_SOD-123, F.Cu at (229.2, 96.4)
- added D2: B5819W_SL, Diode_SMD:D_SOD-123, F.Cu at (275.6, 58.3)
- added D6: B5819W_SL, Diode_SMD:D_SOD-123, F.Cu at (266.3, 83.5)
- added D7: B5819W_SL, Diode_SMD:D_SOD-123, F.Cu at (281.3, 58.3)
- added FID2: Fiducial, Fiducial:Fiducial_0.5mm_Mask1.5mm, F.Cu at (184.8, 122.7)
- added Q3: IRFZ24NPBF, Package_TO_SOT_THT:TO-247-3_Vertical, F.Cu at (126.1, 122.7)
- added R1: 1k, Resistor_SMD:R_0603_1608Metric, F.Cu at (244.7, 115.9)
- added R12: 470, Resistor_SMD:R_0603_1608Metric, F.Cu at (293.6, 61.9)
- added R13: 10k, Resistor_SMD:R_0603_1608Metric, F.Cu at (233.9, 120.9)
- added R14: X, Resistor_THT:R_Axial_DIN0207_L6.3mm_D2.5mm_P10.16mm_Horizontal, F.Cu at (274.3, 54.6)
- added R15: 10k, Resistor_SMD:R_0603_1608Metric, F.Cu at (261.6, 105.7)
- added R16: 470, Resistor_SMD:R_0603_1608Metric, F.Cu at (241.9, 120.9)
- added R17: 100k, Resistor_SMD:R_0603_1608Metric, F.Cu at (305.3, 56.4)
- added R18: 10k, Resistor_SMD:R_0603_1608Metric, F.Cu at (286.6, 78.3)
- added R19: 10k, Resistor_SMD:R_0603_1608Metric, F.Cu at (291.5, 71.9)
- added R2: DNP, Resistor_SMD:R_0603_1608Metric_Pad0.98x0.95mm_HandSolder, F.Cu at (239.1, 87.7)
- added R20: 10k, Resistor_SMD:R_0603_1608Metric, F.Cu at (292.0, 66.9)
- added R21: 100k, Resistor_SMD:R_0603_1608Metric, F.Cu at (293.6, 59.4)
- added R22: 10k, Resistor_SMD:R_0603_1608Metric, F.Cu at (240.7, 118.4)
- added R24: 1k, Resistor_SMD:R_0603_1608Metric, F.Cu at (244.7, 118.4)
- added R27: 100, Resistor_SMD:R_0603_1608Metric, F.Cu at (265.4, 96.5)
- added R3: 10k, Resistor_SMD:R_0603_1608Metric, F.Cu at (284.0, 68.2)
- added R36: 10k, Resistor_SMD:R_0603_1608Metric, F.Cu at (279.2, 84.0)
- added R37: 10k, Resistor_SMD:R_0603_1608Metric, F.Cu at (293.6, 64.4)
- added R39: 100k, Resistor_SMD:R_0603_1608Metric, F.Cu at (264.5, 89.0)
- added R40: 100, Resistor_SMD:R_0603_1608Metric, F.Cu at (229.9, 120.9)
- added R42: 10k, Resistor_SMD:R_0603_1608Metric, F.Cu at (282.6, 76.0)
- added R43: 20k, Resistor_SMD:R_0603_1608Metric, F.Cu at (289.6, 63.4)
- added R44: 1Meg, Resistor_SMD:R_0603_1608Metric, F.Cu at (274.5, 76.4)
- added R45: 10k, Resistor_SMD:R_0603_1608Metric, F.Cu at (301.7, 58.9)
- added R46: 10k, Resistor_SMD:R_0603_1608Metric, F.Cu at (226.1, 131.1)
- added R47: 100m, Resistor_SMD:R_0805_2012Metric, F.Cu at (260.3, 83.3)
- added R48: 20k, Resistor_SMD:R_0603_1608Metric, F.Cu at (283.5, 73.2)
- added R49: 10k, Resistor_SMD:R_0603_1608Metric, F.Cu at (292.0, 69.4)
- added R5: 1Meg, Resistor_SMD:R_0603_1608Metric, F.Cu at (230.1, 131.1)
- added R50: 10k, Resistor_SMD:R_0603_1608Metric, F.Cu at (296.0, 69.4)
- added R51: 1k, Resistor_SMD:R_0603_1608Metric, F.Cu at (297.7, 53.9)
- added R52: 1k, Resistor_SMD:R_0603_1608Metric, F.Cu at (279.2, 78.9)
- added R53: 1k, Resistor_SMD:R_0603_1608Metric, F.Cu at (230.5, 125.9)
- added R54: 1k, Resistor_SMD:R_0603_1608Metric, F.Cu at (289.6, 60.9)
- added R55: 100, Resistor_SMD:R_0603_1608Metric, F.Cu at (269.7, 94.0)
- added R56: 20k, Resistor_SMD:R_0603_1608Metric, F.Cu at (264.5, 86.4)
- added R57: 20k, Resistor_SMD:R_0603_1608Metric, F.Cu at (284.0, 70.7)
- added R58: 10k, Resistor_SMD:R_0603_1608Metric, F.Cu at (275.2, 84.0)
- added R59: 100m, Resistor_SMD:R_0805_2012Metric, F.Cu at (214.4, 132.8)
- added R60: 100m, Resistor_SMD:R_0805_2012Metric, F.Cu at (217.5, 129.2)
- added R61: 100m, Resistor_SMD:R_0805_2012Metric, F.Cu at (210.0, 132.8)
- added R62: 100m, Resistor_SMD:R_0805_2012Metric, F.Cu at (236.5, 116.1)
- added R63: DNP, Resistor_SMD:R_0603_1608Metric_Pad0.98x0.95mm_HandSolder, F.Cu at (279.3, 73.5)
- added R64: 100k, Resistor_SMD:R_0603_1608Metric, F.Cu at (283.2, 80.8)
- added R65: 100k, Resistor_SMD:R_0603_1608Metric, F.Cu at (271.2, 83.7)
- added R66: 1k, Resistor_SMD:R_0603_1608Metric, F.Cu at (288.0, 65.9)
- added R67: 1k, Resistor_SMD:R_0603_1608Metric, F.Cu at (248.8, 118.4)
- added R68: 100k, Resistor_SMD:R_0603_1608Metric, F.Cu at (229.9, 123.4)
- added R69: 100m, Resistor_SMD:R_0805_2012Metric, F.Cu at (274.9, 73.7)
- added R70: 100m, Resistor_SMD:R_0805_2012Metric, F.Cu at (260.3, 86.2)
- added R71: 100k, Resistor_SMD:R_0603_1608Metric, F.Cu at (276.6, 89.0)
- added R72: 100m, Resistor_SMD:R_0805_2012Metric, F.Cu at (279.8, 68.9)
- added R73: 100m, Resistor_SMD:R_0805_2012Metric, F.Cu at (218.8, 132.2)
- added R74: 100m, Resistor_SMD:R_0805_2012Metric, F.Cu at (221.9, 126.3)
- added R75: 100m, Resistor_SMD:R_0805_2012Metric, F.Cu at (217.5, 126.3)
- added R76: 100m, Resistor_SMD:R_0805_2012Metric, F.Cu at (279.8, 65.9)
- added R77: 100k, Resistor_SMD:R_0603_1608Metric, F.Cu at (248.8, 115.9)
- added R9: 10k, Resistor_SMD:R_0603_1608Metric, F.Cu at (301.7, 63.9)
- added SW4: SW_SPST, SamacSys_Parts:PTS526SK15SMTR2LFS, F.Cu at (231.9, 90.6)
- added U12: 1602_LCD_I2C, Z_mycustom_footprint_lib:1602 LCD I2C, F.Cu at (78.5, 89.5)
- added U13: LM4040DBZ-2.0, Package_TO_SOT_SMD:SOT-23, F.Cu at (275.1, 65.4)
- added U14: LM324, Package_SO:SOIC-14_3.9x8.7mm_P1.27mm, F.Cu at (255.4, 109.5)
- C11: value 47u -> 10u; footprint Capacitor_THT:CP_Radial_D6.3mm_P2.50mm -> Capacitor_SMD:C_0603_1608Metric
- C12: value 47u -> 47n; footprint Capacitor_THT:CP_Radial_D6.3mm_P2.50mm -> Capacitor_SMD:C_0603_1608Metric
- C15: value 22u -> 100n; footprint Capacitor_SMD:C_0805_2012Metric_Pad1.18x1.45mm_HandSolder -> Capacitor_SMD:C_0603_1608Metric
- C16, C17: value 22u -> 10u; footprint Capacitor_SMD:C_0805_2012Metric_Pad1.18x1.45mm_HandSolder -> Capacitor_SMD:C_0603_1608Metric
- C19: value 100n -> 10u; footprint Capacitor_SMD:C_0603_1608Metric_Pad1.08x0.95mm_HandSolder -> Capacitor_SMD:C_0603_1608Metric
- C21: value 4.7u -> 100n; footprint Capacitor_SMD:C_0603_1608Metric_Pad1.08x0.95mm_HandSolder -> Capacitor_SMD:C_0603_1608Metric
- D4: value D_Shockley -> B5819W_SL; footprint Diode_THT:D_DO-15_P5.08mm_Vertical_KathodeUp -> Diode_SMD:D_SOD-123
- FID3: value Fiducial -> trash; footprint Fiducial:Fiducial_0.5mm_Mask1.5mm -> Symbol:WEEE-Logo_4.2x6mm_SilkScreen
- J3: value INPUT -> Input
- J4: value probe -> Precision_output; footprint Connector_PinSocket_2.54mm:PinSocket_1x02_P2.54mm_Vertical -> Connector_PinHeader_2.54mm:PinHeader_1x02_P2.54mm_Vertical
- J7: value Conn_01x03 -> Conn_02x04_Odd_Even; footprint Connector_PinHeader_2.54mm:PinHeader_1x03_P2.54mm_Vertical -> Connector_PinHeader_2.54mm:PinHeader_2x04_P2.54mm_Vertical
- J8: value Out -> INPUT
- J9: value Conn_01x03 -> HOLE; footprint Connector_PinHeader_2.54mm:PinHeader_1x03_P2.54mm_Vertical -> Connector_PinSocket_2.54mm:PinSocket_1x01_P2.54mm_Vertical
- R23, R25: value 1Meg -> 1k; footprint Resistor_SMD:R_0603_1608Metric_Pad0.98x0.95mm_HandSolder -> Resistor_SMD:R_0603_1608Metric
- R26: value DNP -> 1k; footprint Resistor_SMD:R_0603_1608Metric_Pad0.98x0.95mm_HandSolder -> Resistor_SMD:R_0603_1608Metric
- R28: value 1Meg -> 10k; footprint Resistor_SMD:R_0603_1608Metric_Pad0.98x0.95mm_HandSolder -> Resistor_SMD:R_0603_1608Metric
- R29: value 180k -> 20k; footprint Resistor_SMD:R_0603_1608Metric_Pad0.98x0.95mm_HandSolder -> Resistor_SMD:R_0603_1608Metric
- R30: value 470 -> 100k; footprint Resistor_SMD:R_0603_1608Metric_Pad0.98x0.95mm_HandSolder -> Resistor_SMD:R_0603_1608Metric
- R31, R33, R34, R35: footprint Resistor_SMD:R_0603_1608Metric_Pad0.98x0.95mm_HandSolder -> Resistor_SMD:R_0603_1608Metric
- R32: value 470 -> 10k; footprint Resistor_SMD:R_0603_1608Metric_Pad0.98x0.95mm_HandSolder -> Resistor_SMD:R_0603_1608Metric
- R41: value 1R -> 1k; footprint Resistor_THT:R_Axial_Power_L50.0mm_W9.0mm_P55.88mm -> Resistor_SMD:R_0603_1608Metric
- R6: value 1R -> DNP; footprint Resistor_THT:R_Axial_Power_L50.0mm_W9.0mm_P55.88mm -> Resistor_SMD:R_0603_1608Metric_Pad0.98x0.95mm_HandSolder; moved to F.Cu
- R7: value 1R -> 1Meg; footprint Resistor_THT:R_Axial_Power_L50.0mm_W9.0mm_P55.88mm -> Resistor_SMD:R_0603_1608Metric
- R8: value X -> 180k; footprint Resistor_THT:R_Axial_DIN0207_L6.3mm_D2.5mm_P10.16mm_Horizontal -> Resistor_SMD:R_0603_1608Metric_Pad0.98x0.95mm_HandSolder
- SW1: value SW_SPDT -> SW_SPST; footprint Z_mycustom_footprint_lib:SPDT switch 2mm -> SamacSys_Parts:PTS526SK15SMTR2LFS
- SW2: value RotaryEncoder_Switch -> SW_SPDT; footprint Z_mycustom_footprint_lib:PEC12R4230FS0024 -> Z_mycustom_footprint_lib:SPDT switch 2mm
- SW3: value SW_SPDT -> RotaryEncoder_Switch; footprint Z_mycustom_footprint_lib:SPDT switch 2mm -> Z_mycustom_footprint_lib:PEC12R4230FS0024
- U1: value 1043 -> LM358; footprint SamacSys_Parts:1043 -> Package_SO:SOIC-8_3.9x4.9mm_P1.27mm; moved to F.Cu
- U11: value LM2902 -> 1043; footprint Package_SO:SOIC-14_3.9x8.7mm_P1.27mm -> SamacSys_Parts:1043
- U4: value STM32L010K4T6 -> TPS63020DSJR; footprint Package_QFP:LQFP-32_7x7mm_P0.8mm -> Z_mycustom_footprint_lib:TPS63020
- U5: value 1602_LCD_I2C -> ESP32-S3-WROOM-1; footprint Z_mycustom_footprint_lib:1602 LCD I2C -> Espressif:ESP32-S3-WROOM-1
- U6: value LM324A -> DMG9933USD-13; footprint Package_SO:SOIC-14_3.9x8.7mm_P1.27mm -> Package_SO:SOIC-8_3.9x4.9mm_P1.27mm
- U7: value TPS63020DSJR -> LM324; footprint Z_mycustom_footprint_lib:TPS63020 -> Package_SO:SOIC-14_3.9x8.7mm_P1.27mm
- U8: value AP3012KTR-G1 -> LM324; footprint Package_TO_SOT_SMD:SOT-23-5_HandSoldering -> Package_SO:SOIC-14_3.9x8.7mm_P1.27mm
- U9: value DMG9933USD-13 -> TPS61040DBV; footprint Package_SO:SOIC-8_3.9x4.9mm_P1.27mm -> Package_TO_SOT_SMD:SOT-23-5
- moved J9 231.3 mm to (275.0, 69.9)
- moved U11 210.7 mm to (76.5, 56.2), turned to -90 degrees
- moved U6 184.8 mm to (268.3, 76.7)
- moved R33 172.7 mm to (305.7, 58.9)
- moved J3 171.0 mm to (115.2, 172.8)
- moved J8 169.7 mm to (104.0, 172.8)
- moved R34 167.3 mm to (293.2, 56.9)
- moved R35 166.9 mm to (297.6, 64.4)
- moved R26 165.5 mm to (301.3, 56.4)
- moved J4 162.2 mm to (255.8, 84.1), turned to 0 degrees
- moved R31 161.4 mm to (305.7, 53.9)
- moved C15 159.8 mm to (287.5, 73.2)
- moved C21 156.7 mm to (297.6, 61.9)
- moved U10 156.2 mm to (280.7, 62.2)
- moved R29 156.0 mm to (301.7, 61.4)
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Connections:
- C11 pad 1: Net-(C11-Pad1) -> GND
- C11 pad 2: -VDC -> +VDC
- C12 pad 1: -VDC -> Net-(C12-Pad1)
- C15 pad 1: +3V3 -> +12V
- C17 pad 1: +VDC -> +3V3
- C19 pad 1: Net-(C19-Pad1) -> +5V
- C21 pad 1: +BATT -> +12V
- C21 pad 2: GND -> -VDC
- J3 pad 1: LOAD -> GND
- J3 pad 2: GND -> Net-(R45-Pad2)
- J4 pad 1: Net-(J4-Pad1) -> GND
- J7 pad 1: GND -> LOAD_VOLTAGE
- J7 pad 3: +12V -> LOAD_VOLTAGE
- J8 pad 1: GND -> LOAD
- J8 pad 2: Net-(J8-Pad2) -> GND
- J9 pad 1: Net-(J9-Pad1) -> -VDC
- R23 pad 1: -VDC -> PWM_Signal_Sink
- R23 pad 2: GND -> Net-(C24-Pad1)
- R25 pad 1: +3V3 -> Net-(R25-Pad1)
- R25 pad 2: /FB_3V3 -> Net-(C26-Pad1)
- R26 pad 1: +3V3 -> ADC_REF
- R26 pad 2: /FB_3V3 -> +3.3VA
- R28 pad 1: +3V3 -> ADC_Batery
- R28 pad 2: /PG_3V3 -> +VDC
- R29 pad 1: /FB_3V3 -> Net-(R29-Pad1)
- R29 pad 2: GND -> Net-(R25-Pad1)
- R30 pad 1: Net-(D3-Pad1) -> GND
- R30 pad 2: Net-(IC1-Pad3) -> Net-(R27-Pad2)
- R31 pad 2: Net-(IC1-Pad8) -> /SW_OUT
- R32 pad 1: Net-(D5-Pad1) -> GND
- R32 pad 2: Net-(IC1-Pad4) -> Net-(R29-Pad1)
- R33 pad 1: /Set_charge_current -> Net-(Q4-Pad1)
- R33 pad 2: GND -> ADC_Batery
- R34 pad 2: /batt_protection -> Net-(TH1-Pad2)
- R35 pad 1: GND -> Net-(Q3-Pad3)
- R35 pad 2: +5V -> Net-(C28-Pad1)
- R41 pad 1: Net-(J11-Pad2) -> unconnected-(R41-Pad1)
- R41 pad 2: Net-(Q5-Pad1) -> unconnected-(R41-Pad2)
- R6 pad 1: Net-(J4-Pad1) -> +3V3
- R6 pad 2: GND -> /FB_3V3
- R7 pad 1: Net-(J4-Pad2) -> /PG_3V3
- R7 pad 2: GND -> +3V3
- R8 pad 1: Net-(J5-Pad2) -> /FB_3V3
- R8 pad 2: LOAD -> GND
- SW1 pad 2: Net-(C4-Pad1) -> /EN
- SW2 pad MH: GND -> (no net)
- SW3 pad MH: (no net) -> GND
- TH1 pad 2: Net-(R24-Pad1) -> Net-(TH1-Pad2)
- U1 pad 1: +BATT -> /PWM_pump
- U1 pad 2: GND -> /fb__pump
- U11 pad 1: ADC_IN8 -> +BATT
- U11 pad 2: ADC_IN8 -> GND
- U4 pad 1: +3V3 -> Net-(SW2-Pad1)
- U4 pad 10: SPI_SS -> +VDC
- U4 pad 11: SPI_CLK -> +VDC
- U4 pad 12: SPI_MOSI -> /EN_3V3
- U4 pad 13: SPI_MISO -> Net-(SW2-Pad1)
- U4 pad 14: ADC_IN8 -> /PG_3V3
- U4 pad 2: unconnected-(U4-Pad2) -> GND
- U4 pad 3: unconnected-(U4-Pad3) -> /FB_3V3
- U4 pad 4: Net-(C4-Pad1) -> +3V3
- U4 pad 5: unconnected-(U4-Pad5) -> +3V3
- U4 pad 6: CLOCK_in -> Net-(L2-Pad2)
- U4 pad 7: ADC_IN1 -> Net-(L2-Pad2)
- U4 pad 8: SYS_wakeup3 -> Net-(L2-Pad1)
- U4 pad 9: ADC_IN3 -> Net-(L2-Pad1)
- U6 pad 1: Net-(J8-Pad2) -> +BATT
- U6 pad 2: Net-(J9-Pad2) -> /batt_protection
- U6 pad 3: Net-(J7-Pad2) -> +VDC
- U6 pad 4: +12V -> +5V
- U6 pad 5: Net-(C9-Pad1) -> /Drains
- U6 pad 6: Net-(R17-Pad1) -> /Drains
- U6 pad 7: Net-(R17-Pad1) -> /Drains
- U6 pad 8: Net-(R16-Pad1) -> /Drains
- U7 pad 1: Net-(C19-Pad1) -> Net-(R24-Pad1)
- U7 pad 10: +VDC -> Net-(R45-Pad1)
- U7 pad 11: +VDC -> -VDC
- U7 pad 12: /EN_3V3 -> Net-(TH1-Pad2)
- U7 pad 13: Net-(C19-Pad1) -> ADC_heatsink
- U7 pad 14: /PG_3V3 -> ADC_heatsink
- U7 pad 2: GND -> Net-(R24-Pad1)
- U7 pad 3: /FB_3V3 -> Net-(C24-Pad1)
- U7 pad 4: +3V3 -> +12V
- U7 pad 5: +3V3 -> Net-(C25-Pad1)
- U7 pad 6: Net-(L2-Pad2) -> Net-(R29-Pad1)
- U7 pad 7: Net-(L2-Pad2) -> Net-(R25-Pad1)
- U7 pad 8: Net-(L2-Pad1) -> ADC_Source_current
- U7 pad 9: Net-(L2-Pad1) -> Net-(R49-Pad2)
- U8 pad 1: Net-(L1-Pad1) -> Net-(R27-Pad2)
- U8 pad 2: GND -> Net-(R27-Pad2)
- U8 pad 3: Net-(R11-Pad2) -> Net-(C26-Pad1)
- U8 pad 4: Net-(R12-Pad1) -> +12V
- U8 pad 5: +VDC -> Net-(R71-Pad1)
- U9 pad 1: +BATT -> Net-(D7-Pad2)
- U9 pad 2: /batt_protection -> GND
- U9 pad 3: +VDC -> Net-(R63-Pad2)
- U9 pad 4: +5V -> +VDC
- U9 pad 5: /Drains -> +VDC
Other:
- board size 100 x 100 mm -> 100 x 141.4 mm

Commit message: g
Parts:
- removed C11, C16, C17, C4, C5: 10u, Capacitor_SMD:C_0603_1608Metric
- removed C12, C14, C24, C25, C26, C28, C31, C32, C33, C34: 47n, Capacitor_SMD:C_0603_1608Metric
- removed C15, C18, C22, C27, C3: 100n, Capacitor_SMD:C_0603_1608Metric
- removed D2, D6, D7: B5819W_SL, Diode_SMD:D_SOD-123
- removed J7: Conn_02x04_Odd_Even, Connector_PinHeader_2.54mm:PinHeader_2x04_P2.54mm_Vertical
- removed R14: X, Resistor_THT:R_Axial_DIN0207_L6.3mm_D2.5mm_P10.16mm_Horizontal
- removed R15, R22, R28, R32, R33, R34, R35, R36, R37, R42, R45, R46, R49, R50, R58: 10k, Resistor_SMD:R_0603_1608Metric
- removed R17, R21, R30, R39, R64, R65, R68, R71, R77: 100k, Resistor_SMD:R_0603_1608Metric
- removed R23, R24, R25, R26, R41, R51, R52, R53, R54, R66, R67: 1k, Resistor_SMD:R_0603_1608Metric
- removed R29, R48, R56, R57: 20k, Resistor_SMD:R_0603_1608Metric
- removed R40: 100, Resistor_SMD:R_0603_1608Metric
- removed R63: DNP, Resistor_SMD:R_0603_1608Metric_Pad0.98x0.95mm_HandSolder
- removed R69, R70: 100m, Resistor_SMD:R_0805_2012Metric
- removed TH1: 68K@25C~5%, Resistor_THT:R_Axial_DIN0204_L3.6mm_D1.6mm_P2.54mm_Vertical
- removed U11: 1043, SamacSys_Parts:1043
- removed U13: LM4040DBZ-2.0, Package_TO_SOT_SMD:SOT-23
- removed U14, U7, U8: LM324, Package_SO:SOIC-14_3.9x8.7mm_P1.27mm
- removed U9: TPS61040DBV, Package_TO_SOT_SMD:SOT-23-5
- added C20: 1u, Capacitor_SMD:C_0402_1005Metric, F.Cu at (375.2, 106.9)
- added D11: green, LED_SMD:LED_0805_2012Metric, F.Cu at (352.7, 105.4)
- added D12: green, LED_SMD:LED_0805_2012Metric, F.Cu at (352.7, 108.5)
- added FID4: Polarity, Symbol:Polarity_Center_Positive_6mm_SilkScreen, F.Cu at (345.0, 77.4)
- added J5: Li ION cell own power, Z_mycustom_footprint_lib:MYOUNG MY-18650-01, F.Cu at (320.9, 66.2)
- added JP2: Jumper_2_Bridged, Jumper:SolderJumper-2_P1.3mm_Bridged_RoundedPad1.0x1.5mm, F.Cu at (324.1, 108.4)
- added R10: 2k, Resistor_SMD:R_0402_1005Metric, F.Cu at (318.4, 109.6)
- added R4: 470, Resistor_SMD:R_0402_1005Metric, F.Cu at (318.4, 107.6)
- added U15: SRV05-4, Package_TO_SOT_SMD:SOT-23-6, F.Cu at (314.3, 103.8)
- added U3: ESP32-S3-WROOM-1, Espressif:ESP32-S3-WROOM-1, F.Cu at (322.1, 90.5)
- C1: value 100n -> 1u; footprint Capacitor_SMD:C_0603_1608Metric -> Capacitor_SMD:C_0402_1005Metric
- C2: value 10u -> 1u; footprint Capacitor_SMD:C_0603_1608Metric -> Capacitor_SMD:C_0402_1005Metric
- C30: value 100n -> 10u
- C7: value 10u -> 100n
- J4: value Precision_output -> Jack-DC; footprint Connector_PinHeader_2.54mm:PinHeader_1x02_P2.54mm_Vertical -> Connector_BarrelJack:BarrelJack_Wuerth_6941xx301002
- R1: value 1k -> 15-16k
- R2: value DNP -> 1k; footprint Resistor_SMD:R_0603_1608Metric_Pad0.98x0.95mm_HandSolder -> Resistor_SMD:R_0805_2012Metric
- R43: value 20k -> 1k; footprint Resistor_SMD:R_0603_1608Metric -> Resistor_SMD:R_0805_2012Metric
- R44: value 1Meg -> 1k; footprint Resistor_SMD:R_0603_1608Metric -> Resistor_SMD:R_0805_2012Metric
- U1: value LM358 -> AD5337; footprint Package_SO:SOIC-8_3.9x4.9mm_P1.27mm -> Package_SO:MSOP-8_3x3mm_P0.65mm
- U2: value D1213A-02SM -> AD8001AR; footprint Package_TO_SOT_SMD:SOT-23-5_HandSoldering -> Package_SO:SOIC-8_3.9x4.9mm_P1.27mm
- U5: value ESP32-S3-WROOM-1 -> CJ431; footprint Espressif:ESP32-S3-WROOM-1 -> Package_TO_SOT_SMD:SOT-23
- moved D4 209.0 mm to (374.1, 78.9)
- moved FID1 193.8 mm to (364.4, 77.3)
- moved U4 163.2 mm to (371.9, 98.8)
- moved IC1 156.3 mm to (336.2, 99.8)
- moved D3 156.3 mm to (373.6, 91.2)
- moved R61 155.4 mm to (361.9, 100.4)
- moved C8 152.8 mm to (373.6, 82.4)
- moved R75 151.1 mm to (366.4, 100.4)
- moved F1 148.2 mm to (336.1, 104.6)
- moved R60 147.9 mm to (361.9, 97.4)
- moved R74 147.3 mm to (366.4, 97.4)
- moved D1 146.4 mm to (374.1, 75.5)
- moved U1 145.2 mm to (346.8, 106.2)
- moved R59 145.0 mm to (357.5, 109.2)
- moved R73 144.9 mm to (361.9, 109.2)
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Connections:
- C1 pad 1: +VDC -> GND
- C1 pad 2: GND -> +3V3
- C2 pad 1: Net-(C2-Pad1) -> GND
- C2 pad 2: Net-(C2-Pad2) -> REF_2v5
- C29 pad 1: unconnected-(C29-Pad1) -> +3V3
- C29 pad 2: unconnected-(C29-Pad2) -> GND
- C30 pad 1: unconnected-(C30-Pad1) -> +3V3
- C30 pad 2: unconnected-(C30-Pad2) -> GND
- C7 pad 1: GND -> /EN
- C7 pad 2: /EN -> GND
- J4 pad 1: GND -> LOAD
- J4 pad 2: Net-(J4-Pad2) -> GND
- Q3 pad 3: Net-(Q3-Pad3) -> Net-(Q3-S)
- R1 pad 1: Net-(C3-Pad1) -> GND
- R1 pad 2: /PWM_pump -> Net-(U2--)
- R2 pad 1: /PWM_pump -> Net-(U2--)
- R2 pad 2: Net-(C3-Pad1) -> Net-(Q3-S)
- R43 pad 1: unconnected-(R43-Pad1) -> Net-(D11-K)
- R43 pad 2: unconnected-(R43-Pad2) -> Net-(JP2-B)
- R44 pad 1: unconnected-(R44-Pad1) -> Net-(D12-K)
- R44 pad 2: unconnected-(R44-Pad2) -> Net-(JP2-B)
- R47 pad 1: Net-(Q3-Pad3) -> Net-(Q3-S)
- R55 pad 2: Net-(R55-Pad2) -> unconnected-(R55-Pad2)
- R59 pad 1: Net-(Q3-Pad3) -> Net-(Q3-S)
- R60 pad 1: Net-(Q3-Pad3) -> Net-(Q3-S)
- R61 pad 1: Net-(Q3-Pad3) -> Net-(Q3-S)
- R62 pad 1: Net-(Q3-Pad3) -> Net-(Q3-S)
- U1 pad 1: /PWM_pump -> +3V3
- U1 pad 2: /fb__pump -> /DAC1
- U1 pad 3: Net-(C3-Pad1) -> /DAC2
- U1 pad 4: GND -> REF_2v5
- U1 pad 5: /PWM_pump -> GND
- U1 pad 6: Net-(C2-Pad1) -> SDA
- U1 pad 7: Net-(C2-Pad1) -> SCL
- U1 pad 8: +VDC -> GND
- U2 pad 2: GND -> Net-(U2--)
- U2 pad 3: D- -> /DAC1
- U2 pad 4: D+ -> unconnected-(U2-V--Pad4)
- U2 pad 5: VBUS -> unconnected-(U2-NC-Pad5)
- U5 pad 1: GND -> REF_2v5
- U5 pad 2: +3V3 -> REF_2v5
- U5 pad 3: /EN -> GND
