File: Small_load_V1/Small_load_V1.kicad_pcb (KiCad board)
At the start: 2 copper layers, 100 x 141.4 mm, 86 parts, among them IC1 MCP73834T-FCI_UN, J1 USB_B, J12 LOAD, J3 Input, J4 Jack-DC, J5 Li ION cell own power, J8 INPUT, J9 HOLE, Q3 IRFZ24NPBF, Q5 Q_PMOS_DGS, SW1 SW_SPST, SW2 SW_SPDT, SW3 RotaryEncoder_Switch, SW4 SW_SPST, U1 AD5337, U10 APX810S05, U12 1602_LCD_I2C, U15 SRV05-4, U2 AD8001AR, U3 ESP32-S3-WROOM-1, U4 TPS63020DSJR, U5 CJ431, U6 DMG9933USD-13

Commit message: l
Parts:
- removed J12: LOAD, TerminalBlock:TerminalBlock_Altech_AK300-2_P5.00mm
- removed L2: 1.5u, Inductor_SMD:L_Wuerth_MAPI-3012
- removed R55: 100, Resistor_SMD:R_0603_1608Metric
- removed R59, R60, R61, R62, R72, R73, R74, R75, R76: 100m, Resistor_SMD:R_0805_2012Metric
- removed SW2: SW_SPDT, Z_mycustom_footprint_lib:SPDT switch 2mm
- added C11: 10u, Capacitor_SMD:C_0603_1608Metric, F.Cu at (-46.3, 68.9)
- added C12: 10u, Capacitor_SMD:C_0603_1608Metric, F.Cu at (-46.3, 71.4)
- added C14: 10u, Capacitor_SMD:C_0603_1608Metric, F.Cu at (-46.3, 76.4)
- added C15: 10u, Capacitor_SMD:C_0603_1608Metric, F.Cu at (-46.3, 78.9)
- added C16: 10u, Capacitor_SMD:C_0603_1608Metric, F.Cu at (-46.3, 81.4)
- added C17: 10u, Capacitor_SMD:C_0603_1608Metric, F.Cu at (-42.3, 61.4)
- added C18: 10u, Capacitor_SMD:C_0603_1608Metric, F.Cu at (-42.3, 63.9)
- added C22: 10u, Capacitor_SMD:C_0603_1608Metric, F.Cu at (-42.3, 66.4)
- added C24: 10u, Capacitor_SMD:C_0603_1608Metric, F.Cu at (-42.3, 68.9)
- added C25: 10u, Capacitor_SMD:C_0603_1608Metric, F.Cu at (-42.3, 71.4)
- added C26: 10u, Capacitor_SMD:C_0603_1608Metric, F.Cu at (-42.3, 73.9)
- added C27: 10u, Capacitor_SMD:C_0603_1608Metric, F.Cu at (-42.3, 76.4)
- added C28: 10u, Capacitor_SMD:C_0603_1608Metric, F.Cu at (-42.3, 78.9)
- added C3: 100p, Capacitor_SMD:C_0603_1608Metric, F.Cu at (273.0, 132.9)
- added C31: 10u, Capacitor_SMD:C_0603_1608Metric, F.Cu at (-42.3, 81.4)
- added C32: 10u, Capacitor_SMD:C_0603_1608Metric, F.Cu at (-38.3, 61.4)
- added C33: 10u, Capacitor_SMD:C_0603_1608Metric, F.Cu at (-38.3, 63.9)
- added C34: 10u, Capacitor_SMD:C_0603_1608Metric, F.Cu at (-38.3, 66.4)
- added C35: 10u, Capacitor_SMD:C_0603_1608Metric, F.Cu at (-38.3, 68.9)
- added C36: 10u, Capacitor_SMD:C_0603_1608Metric, F.Cu at (-38.3, 71.4)
- added C37: 10u, Capacitor_SMD:C_0603_1608Metric, F.Cu at (-38.3, 73.9)
- added C38: 10u, Capacitor_SMD:C_0603_1608Metric, F.Cu at (-38.3, 76.4)
- added C39: 10u, Capacitor_SMD:C_0603_1608Metric, F.Cu at (-38.3, 78.9)
- added C4: 1u, Capacitor_SMD:C_0402_1005Metric, F.Cu at (-30.9, 90.1)
- added C40: 10u, Capacitor_SMD:C_0603_1608Metric, F.Cu at (-38.3, 81.4)
- added C41: 10u, Capacitor_SMD:C_0603_1608Metric, F.Cu at (-34.3, 61.4)
- added C42: 10u, Capacitor_SMD:C_0603_1608Metric, F.Cu at (-34.3, 63.9)
- added C43: 10u, Capacitor_SMD:C_0603_1608Metric, F.Cu at (-34.3, 66.4)
- added C44: 10u, Capacitor_SMD:C_0603_1608Metric, F.Cu at (-34.3, 68.9)
- added C45: 10u, Capacitor_SMD:C_0603_1608Metric, F.Cu at (-34.3, 71.4)
- added C46: 10u, Capacitor_SMD:C_0603_1608Metric, F.Cu at (-34.3, 73.9)
- added C47: 10u, Capacitor_SMD:C_0603_1608Metric, F.Cu at (-34.3, 76.4)
- added C48: 10u, Capacitor_SMD:C_0603_1608Metric, F.Cu at (-34.3, 78.9)
- added C49: 10u, Capacitor_SMD:C_0603_1608Metric, F.Cu at (-34.3, 81.4)
- added C5: 100p, Capacitor_SMD:C_0603_1608Metric, F.Cu at (273.0, 135.4)
- added C50: 10u, Capacitor_SMD:C_0603_1608Metric, F.Cu at (-30.3, 61.4)
- added C51: 10u, Capacitor_SMD:C_0603_1608Metric, F.Cu at (-30.3, 63.9)
- added C52: 10u, Capacitor_SMD:C_0603_1608Metric, F.Cu at (-30.3, 66.4)
- added C53: 10u, Capacitor_SMD:C_0603_1608Metric, F.Cu at (-30.3, 68.9)
- added C54: 10u, Capacitor_SMD:C_0603_1608Metric, F.Cu at (-30.3, 71.4)
- added C55: 10u, Capacitor_SMD:C_0603_1608Metric, F.Cu at (-30.3, 73.9)
- added FID5: Polarity, Symbol:Polarity_Center_Positive_6mm_SilkScreen, F.Cu at (301.0, 96.7)
- added J2: Jack-DC, Connector_BarrelJack:BarrelJack_Wuerth_6941xx301002, F.Cu at (210.2, 124.9)
- added J6: Conn_01x08, Connector_PinHeader_2.54mm:PinHeader_1x08_P2.54mm_Vertical, F.Cu at (-46.0, 85.0)
- added Q1: IRF9540N, Package_TO_SOT_THT:TO-220-3_Vertical, F.Cu at (119.3, 101.7)
- added Q2: AGM420MC, Package_SO:SOIC-8_3.9x4.9mm_P1.27mm, F.Cu at (-52.5, 63.3)
- added Q4: AGM420MC, Package_SO:SOIC-8_3.9x4.9mm_P1.27mm, F.Cu at (-52.5, 69.8)
- added Q6: AGM420MC, Package_SO:SOIC-8_3.9x4.9mm_P1.27mm, F.Cu at (-52.5, 82.7)
- added Q7: AGM420MC, Package_SO:SOIC-8_3.9x4.9mm_P1.27mm, F.Cu at (-52.5, 89.1)
- added Q8: AGM420MC, Package_SO:SOIC-8_3.9x4.9mm_P1.27mm, F.Cu at (-52.5, 95.6)
- added Q9: AGM420MC, Package_SO:SOIC-8_3.9x4.9mm_P1.27mm, F.Cu at (-52.5, 102.0)
- added R11: 50m, Resistor_THT:R_Axial_DIN0516_L15.5mm_D5.0mm_P20.32mm_Horizontal, F.Cu at (290.4, 83.3)
- added R14: 2k, Resistor_SMD:R_0402_1005Metric, F.Cu at (307.7, 60.2)
- added U7: AD8001AR, Package_SO:SOIC-8_3.9x4.9mm_P1.27mm, F.Cu at (303.9, 120.0)
- added U8: AD8001AR, Package_SO:SOIC-8_3.9x4.9mm_P1.27mm, F.Cu at (303.9, 126.5)
- C10, C8, C9: value 22u -> 10u; footprint Capacitor_SMD:C_0805_2012Metric -> Capacitor_SMD:C_0603_1608Metric
- C13: value 100n -> 10u
- Q5: value Q_PMOS_DGS -> AGM420MC; footprint Package_TO_SOT_THT:TO-247-3_Vertical -> Package_SO:SOIC-8_3.9x4.9mm_P1.27mm
- R47: value 100m -> 50m; footprint Resistor_SMD:R_0805_2012Metric -> Resistor_THT:R_Axial_DIN0516_L15.5mm_D5.0mm_P20.32mm_Horizontal
- R5: value 1Meg -> 100
- R6: value DNP -> 10k; footprint Resistor_SMD:R_0603_1608Metric_Pad0.98x0.95mm_HandSolder -> Resistor_SMD:R_0603_1608Metric
- R7: value 1Meg -> 10k
- R8: value 180k -> 10k; footprint Resistor_SMD:R_0603_1608Metric_Pad0.98x0.95mm_HandSolder -> Resistor_SMD:R_0603_1608Metric
- U4: value TPS63020DSJR -> MCP3208; footprint Z_mycustom_footprint_lib:TPS63020 -> Package_SO:SOIC-16_3.9x9.9mm_P1.27mm
- moved C10 420.5 mm to (-46.3, 66.4)
- moved C9 420.5 mm to (-46.3, 63.9)
- moved C8 420.4 mm to (-46.3, 61.4)
- moved U4 411.5 mm to (-39.5, 88.4)
- moved C2 406.5 mm to (-30.9, 88.1)
- moved C13 403.9 mm to (-46.3, 73.9)
- moved R10 352.7 mm to (-33.8, 90.1)
- moved R4 352.7 mm to (-33.8, 88.1)
- moved J5 299.8 mm to (26.9, 125.1), turned to 90 degrees
- moved U2 239.7 mm to (303.9, 107.1), turned to 0 degrees
- moved J8 223.5 mm to (304.0, 73.1)
- moved J3 202.8 mm to (291.8, 73.1)
- moved J1 196.1 mm to (254.2, 125.6), turned to 0 degrees
- moved Q5 188.9 mm to (-52.5, 76.2), turned to 0 degrees
- moved D1 168.3 mm to (219.1, 141.2)
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Connections:
- C10 pad 1: +3V3 -> Net-(C10-Pad1)
- C10 pad 2: GND -> Net-(C10-Pad2)
- C13 pad 1: Net-(SW2-A) -> Net-(C10-Pad1)
- C13 pad 2: GND -> Net-(C10-Pad2)
- C8 pad 1: GND -> Net-(C10-Pad1)
- C8 pad 2: +VDC -> Net-(C10-Pad2)
- C9 pad 1: +3V3 -> Net-(C10-Pad1)
- C9 pad 2: GND -> Net-(C10-Pad2)
- Q5 pad 1: Net-(Q5-D) -> /Cell_balancer/S4
- Q5 pad 2: Net-(Q5-G) -> unconnected-(Q5A-G-Pad2)
- Q5 pad 3: Net-(J12-Pin_1) -> /Cell_balancer/S5
- R5 pad 1: /FB_3V3 -> Net-(Q1-G)
- R5 pad 2: +3V3 -> Net-(R5-Pad2)
- R6 pad 1: +3V3 -> Net-(U7-+)
- R6 pad 2: /FB_3V3 -> Net-(Q1-D)
- R7 pad 1: /PG_3V3 -> Net-(R14-Pad1)
- R7 pad 2: +3V3 -> Net-(J3-Pin_2)
- R8 pad 1: /FB_3V3 -> GND
- R8 pad 2: GND -> Net-(U7-+)
- U4 pad 1: Net-(SW2-A) -> unconnected-(U4-CH0-Pad1)
- U4 pad 10: +VDC -> unconnected-(U4-~{CS}/SHDN-Pad10)
- U4 pad 11: +VDC -> unconnected-(U4-Din-Pad11)
- U4 pad 12: /EN_3V3 -> unconnected-(U4-Dout-Pad12)
- U4 pad 13: Net-(SW2-A) -> unconnected-(U4-CLK-Pad13)
- U4 pad 14: /PG_3V3 -> GND
- U4 pad 2: GND -> unconnected-(U4-CH1-Pad2)
- U4 pad 3: /FB_3V3 -> unconnected-(U4-CH2-Pad3)
- U4 pad 4: +3V3 -> unconnected-(U4-CH3-Pad4)
- U4 pad 5: +3V3 -> unconnected-(U4-CH4-Pad5)
- U4 pad 6: Net-(L2-Pad2) -> unconnected-(U4-CH5-Pad6)
- U4 pad 7: Net-(L2-Pad2) -> unconnected-(U4-CH6-Pad7)
- U4 pad 8: Net-(L2-Pad1) -> unconnected-(U4-CH7-Pad8)
- U4 pad 9: Net-(L2-Pad1) -> GND
Routing:
- added copper zone on F.Cu, net GND
Other:
- board size 100 x 141.4 mm -> 101 x 101 mm

Commit message: g
Parts:
- removed C13, C14, C15, C16, C17, C18, C22, C23, C24, C25, C26, C27, C28, C31, C32, C33, C34, C35, C36, C37, C38, C39, C40, C41, C42, C43, C44, C45, C46, C47, C48, C49, C50, C51, C52, C53, C54, C55: 10u, Capacitor_SMD:C_0603_1608Metric
- removed IC1: MCP73834T-FCI_UN, SamacSys_Parts:SOP50P490X110-10N
- removed J2: Jack-DC, Connector_BarrelJack:BarrelJack_Wuerth_6941xx301002
- removed J9: HOLE, Connector_PinSocket_2.54mm:PinSocket_1x01_P2.54mm_Vertical
- removed Q8, Q9: AGM420MC, Package_SO:SOIC-8_3.9x4.9mm_P1.27mm
- removed R43, R44: 1k, Resistor_SMD:R_0805_2012Metric
- added C56: 100p, Capacitor_SMD:C_0603_1608Metric, F.Cu at (196.1, 103.3)
- added D2: 1N5819WS, Diode_SMD:D_SOD-323, F.Cu at (324.9, 27.1)
- added FID7: Polarity, Symbol:Polarity_Center_Positive_6mm_SilkScreen, F.Cu at (224.5, 20.1)
- added J10: Jack-DC, Connector_BarrelJack:BarrelJack_Wuerth_6941xx301002, F.Cu at (208.6, 135.8)
- added J11: Input, TerminalBlock:TerminalBlock_Altech_AK300-2_P5.00mm, F.Cu at (204.0, 65.8)
- added Q10: IRFZ24NPBF, Package_TO_SOT_THT:TO-247-3_Vertical, F.Cu at (120.1, 98.8)
- added R15: 100, Resistor_SMD:R_0603_1608Metric, F.Cu at (196.1, 111.3)
- added R17: 10k, Resistor_SMD:R_0603_1608Metric, F.Cu at (191.1, 111.3)
- added R21: 56, Resistor_SMD:R_0603_1608Metric, F.Cu at (328.5, 10.1)
- added R22: 1, Resistor_THT:R_Axial_DIN0516_L15.5mm_D5.0mm_P20.32mm_Horizontal, F.Cu at (226.9, 120.0)
- added R23: 56, Resistor_SMD:R_0603_1608Metric, F.Cu at (328.5, 12.6)
- added R24: 10k, Resistor_SMD:R_0603_1608Metric, F.Cu at (304.0, 35.3)
- added R25: 100, Resistor_SMD:R_0603_1608Metric, F.Cu at (304.0, 37.8)
- added R26: 1k, Resistor_SMD:R_0603_1608Metric, F.Cu at (304.0, 40.3)
- added R28: 1k, Resistor_SMD:R_0603_1608Metric, F.Cu at (304.0, 42.8)
- added R29: 10k, Resistor_SMD:R_0603_1608Metric, F.Cu at (304.0, 45.4)
- added R30: 1k, Resistor_SMD:R_0603_1608Metric, F.Cu at (304.0, 47.9)
- added R32: 10k, Resistor_SMD:R_0603_1608Metric, F.Cu at (304.0, 50.4)
- added R41: 50m, Resistor_THT:R_Axial_DIN0516_L15.5mm_D5.0mm_P20.32mm_Horizontal, F.Cu at (220.3, 120.0)
- added R46: 10k, Resistor_SMD:R_0603_1608Metric, F.Cu at (196.1, 115.3)
- added R48: 10k, Resistor_SMD:R_0603_1608Metric, F.Cu at (193.6, 115.3)
- added R49: 40k2, Resistor_SMD:R_0603_1608Metric, F.Cu at (191.1, 115.3)
- added R50: 2k, Resistor_SMD:R_0402_1005Metric, F.Cu at (185.1, 41.4)
- added R51: 10k, Resistor_SMD:R_0603_1608Metric, F.Cu at (188.6, 115.3)
- added U11: LM324A, Package_SO:SOIC-14_3.9x8.7mm_P1.27mm, F.Cu at (310.2, 39.2)
- added U13: LM324A, Package_SO:SOIC-14_3.9x8.7mm_P1.27mm, F.Cu at (318.7, 39.2)
- added U9: AD8001AR, Package_SO:SOIC-8_3.9x4.9mm_P1.27mm, F.Cu at (187.3, 54.4)
- C10, C9: footprint Capacitor_SMD:C_0603_1608Metric -> Capacitor_SMD:C_1206_3216Metric
- C11: value 10u -> 100p
- C12: footprint Capacitor_SMD:C_0603_1608Metric -> Capacitor_SMD:C_0805_2012Metric
- C19: value 10u -> 1u; footprint Capacitor_SMD:C_0603_1608Metric -> Capacitor_SMD:C_0402_1005Metric
- C5: value 100p -> 100n
- C8: value 10u -> 10u@50V; footprint Capacitor_SMD:C_0603_1608Metric -> Capacitor_SMD:C_0805_2012Metric
- D3: value LED_Small -> 1N5819WS; footprint LED_SMD:LED_0603_1608Metric_Pad1.05x0.95mm_HandSolder -> Diode_SMD:D_SOD-323
- D4: value B5819W_SL -> 1N4007; footprint Diode_SMD:D_SOD-123 -> Diode_THT:D_DO-41_SOD81_P10.16mm_Horizontal
- D5: value LED_Small -> 1N4007; footprint LED_SMD:LED_0603_1608Metric_Pad1.05x0.95mm_HandSolder -> Diode_THT:D_DO-41_SOD81_P10.16mm_Horizontal
- J3: value Input -> Jack-DC; footprint TerminalBlock:TerminalBlock_Altech_AK300-2_P5.00mm -> Connector_BarrelJack:BarrelJack_Wuerth_6941xx301002
- J6: value Conn_01x08 -> Input; footprint Connector_PinHeader_2.54mm:PinHeader_1x08_P2.54mm_Vertical -> TerminalBlock:TerminalBlock_Altech_AK300-2_P5.00mm
- Q1: value IRF9540N -> 2N7002; footprint Package_TO_SOT_THT:TO-220-3_Vertical -> Package_TO_SOT_SMD:SOT-23
- Q2: value AGM420MC -> 2N7002; footprint Package_SO:SOIC-8_3.9x4.9mm_P1.27mm -> Package_TO_SOT_SMD:SOT-23
- Q4, Q6: value AGM420MC -> HYG025N06LS1C2; footprint Package_SO:SOIC-8_3.9x4.9mm_P1.27mm -> Z_mycustom_footprint_lib:DFN-8_(5x6)
- Q5: value AGM420MC -> IRF9540N; footprint Package_SO:SOIC-8_3.9x4.9mm_P1.27mm -> Package_TO_SOT_THT:TO-220-3_Vertical
- Q7: value AGM420MC -> 2N3904; footprint Package_SO:SOIC-8_3.9x4.9mm_P1.27mm -> Package_TO_SOT_THT:TO-92_Inline
- R1: value 15-16k -> 3k
- R10: value 2k -> 1k; footprint Resistor_SMD:R_0402_1005Metric -> Resistor_SMD:R_0603_1608Metric
- R11: value 50m -> 1k; footprint Resistor_THT:R_Axial_DIN0516_L15.5mm_D5.0mm_P20.32mm_Horizontal -> Resistor_SMD:R_0603_1608Metric
- R12: value 470 -> 1k
- R13: value 10k -> 1k; footprint Resistor_SMD:R_0603_1608Metric -> Resistor_THT:R_Axial_DIN0309_L9.0mm_D3.2mm_P5.08mm_Vertical
- R14: value 2k -> 10k; footprint Resistor_SMD:R_0402_1005Metric -> Resistor_SMD:R_0603_1608Metric
- R16: value 470 -> 10k
- R19, R20: value 10k -> 56
- R2: footprint Resistor_SMD:R_0805_2012Metric -> Resistor_SMD:R_0603_1608Metric
- R5: value 100 -> 2k; footprint Resistor_SMD:R_0603_1608Metric -> Resistor_SMD:R_0402_1005Metric
- R6, R8: value 10k -> 1k
- R7: value 10k -> 3k
- U10: value APX810S05 -> AD5337; footprint Package_TO_SOT_SMD:SOT-23 -> Package_SO:MSOP-8_3x3mm_P0.65mm
- U12: footprint Z_mycustom_footprint_lib:1602 LCD I2C -> Z_mycustom_footprint_lib:1602_LCD_mine
- U6: value DMG9933USD-13 -> LM5109BMA
- U7, U8: value AD8001AR -> LM324A; footprint Package_SO:SOIC-8_3.9x4.9mm_P1.27mm -> Package_SO:SOIC-14_3.9x8.7mm_P1.27mm
- moved Q6 381.6 mm to (323.7, 19.1)
- moved Q7 376.8 mm to (321.9, 47.5)
- moved Q4 373.4 mm to (317.4, 19.1)
- moved J6 371.1 mm to (317.6, 10.8)
- moved C12 359.2 mm to (309.9, 24.9)
- moved C8 358.4 mm to (309.9, 21.9)
- moved C9 353.6 mm to (304.8, 22.1)
- moved C10 353.5 mm to (304.8, 25.4)
- moved Q2 287.8 mm to (223.5, 144.7), turned to -90 degrees
- moved C2 265.0 mm to (227.2, 148.6), turned to -90 degrees
- moved C4 262.7 mm to (225.2, 148.6), turned to -90 degrees
- moved U5 258.8 mm to (219.0, 144.7), turned to -90 degrees
- moved C11 239.4 mm to (191.1, 99.3), turned to -90 degrees
- moved U4 232.2 mm to (191.3, 62.8), turned to -90 degrees
- moved R4 227.7 mm to (189.1, 41.4), turned to -90 degrees
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Connections:
- C10 pad 1: Net-(C10-Pad1) -> Net-(Q4-D)
- C10 pad 2: Net-(C10-Pad2) -> GND
- C11 pad 1: Net-(C10-Pad1) -> VLDO_OUT
- C11 pad 2: Net-(C10-Pad2) -> Net-(U7B-+)
- C12 pad 1: Net-(C10-Pad1) -> /buck/HB1
- C12 pad 2: Net-(C10-Pad2) -> Net-(Q4-S)
- C19 pad 1: +5V -> GND
- C19 pad 2: GND -> +3V3
- C5 pad 1: Net-(Q1-D) -> REF_2v5
- C5 pad 2: Net-(U7-+) -> GND
- C8 pad 1: Net-(C10-Pad1) -> GND
- C8 pad 2: Net-(C10-Pad2) -> +15V
- C9 pad 1: Net-(C10-Pad1) -> Net-(Q4-D)
- C9 pad 2: Net-(C10-Pad2) -> GND
- D1 pad 1: +VDC -> /buck/HB1
- D1 pad 2: +5V -> +15V
- D3 pad 2: +5V -> /buck/gate_L1
- D4 pad 1: +VDC -> GND
- D4 pad 2: +5V -> Net-(D4-A)
- D5 pad 1: Net-(D5-K) -> Net-(D4-A)
- D5 pad 2: +5V -> Net-(D5-A)
- J3 pad 1: GND -> Net-(Q4-D)
- J3 pad 2: Net-(J3-Pin_2) -> GND
- J6 pad 2: /Cell_balancer/S1 -> unconnected-(J6-Pin_2-Pad2)
- Q1 pad 1: Net-(Q1-G) -> +3V3
- Q1 pad 2: Net-(Q1-D) -> I2C_SDA_3V3
- Q1 pad 3: Net-(Q1-S) -> I2C_SDA
- Q2 pad 1: /Cell_balancer/S6 -> +3V3
- Q2 pad 2: unconnected-(Q2A-G-Pad2) -> I2C_CLK_3V3
- Q2 pad 3: /Cell_balancer/S7 -> I2C_CLK
- Q4 pad 1: /Cell_balancer/S5 -> Net-(Q4-D)
- Q4 pad 2: unconnected-(Q4A-G-Pad2) -> Net-(Q4-S)
- Q4 pad 3: /Cell_balancer/S6 -> /buck/gate_H1
- Q5 pad 1: /Cell_balancer/S4 -> Net-(Q5-G)
- Q5 pad 2: unconnected-(Q5A-G-Pad2) -> VLDO_OUT
- Q5 pad 3: /Cell_balancer/S5 -> Net-(Q5-S)
- Q6 pad 1: /Cell_balancer/S3 -> Net-(Q4-S)
- Q6 pad 2: unconnected-(Q6A-G-Pad2) -> GND
- Q6 pad 3: /Cell_balancer/S4 -> /buck/gate_L1
- Q7 pad 1: /Cell_balancer/S2 -> GND
- Q7 pad 2: unconnected-(Q7A-G-Pad2) -> Net-(Q7-B)
- Q7 pad 3: /Cell_balancer/S3 -> Net-(Q7-C)
- R10 pad 1: +VDC -> Net-(D12-K)
- R10 pad 2: REF_2v5 -> Net-(JP2-B)
- R11 pad 1: Net-(J3-Pin_2) -> Net-(Q5-S)
- R11 pad 2: Net-(Q1-S) -> Net-(U7D--)
- R12 pad 1: Net-(D3-K) -> /LDO_Vcc
- R12 pad 2: Net-(IC1-STAT1) -> Net-(U7D-+)
- R13 pad 1: GND -> Net-(J2-Pin_5)
- R13 pad 2: Net-(IC1-THERM) -> +3V3
- R14 pad 1: Net-(R14-Pad1) -> I2C_SDA
- R14 pad 2: GND -> +5V
- R16 pad 1: Net-(IC1-STAT2) -> I2C_CLK
- R16 pad 2: Net-(D5-K) -> +5V
- R18 pad 1: GND -> I2C_CLK_3V3
- R18 pad 2: /Set_charge_current -> +3V3
- R19 pad 1: GND -> /buck/HO1
- R19 pad 2: /batt_protection -> Net-(D2-K)
- R2 pad 1: Net-(U2--) -> Net-(Q10-S)
- R2 pad 2: Net-(Q3-S) -> Net-(U9--)
- R20 pad 1: GND -> /buck/gate_H1
- R20 pad 2: +5V -> /buck/HO1
- R4 pad 2: +VDC -> +3V3
- R5 pad 1: Net-(Q1-G) -> +3V3
- R5 pad 2: Net-(R5-Pad2) -> REF_2v5
- R6 pad 1: Net-(U7-+) -> Net-(Q3-S)
- R6 pad 2: Net-(Q1-D) -> Net-(U2--)
- R7 pad 1: Net-(R14-Pad1) -> GND
- R7 pad 2: Net-(J3-Pin_2) -> Net-(U9--)
- R8 pad 1: GND -> Net-(D11-K)
- R8 pad 2: Net-(U7-+) -> Net-(JP2-B)
- U10 pad 1: /batt_protection -> +3V3
- U10 pad 2: GND -> /DAC3
- U10 pad 3: +BATT -> /DAC4
- U6 pad 1: +BATT -> +15V
- U6 pad 2: /batt_protection -> /buck/Phase_A_H
- U6 pad 3: +VDC -> /buck/Phase_A_L
- U6 pad 4: +5V -> GND
- U6 pad 5: /Drains -> /buck/LO1
- U6 pad 6: /Drains -> Net-(Q4-S)
- U6 pad 7: /Drains -> /buck/HO1
- U6 pad 8: /Drains -> /buck/HB1
- U7 pad 1: unconnected-(U7-NC-Pad1) -> (no net)
- U7 pad 2: /DAC2 -> (no net)
- U7 pad 3: Net-(U7-+) -> (no net)
- U7 pad 4: unconnected-(U7-V--Pad4) -> (no net)
- U7 pad 5: unconnected-(U7-NC-Pad5) -> (no net)
- U7 pad 6: Net-(R5-Pad2) -> (no net)
- U7 pad 7: unconnected-(U7-V+-Pad7) -> (no net)
- U7 pad 8: unconnected-(U7-NC-Pad8) -> (no net)
- U8 pad 1: unconnected-(U8-NC-Pad1) -> (no net)
- U8 pad 2: Net-(Q1-S) -> (no net)
- U8 pad 3: Net-(J3-Pin_2) -> (no net)
- U8 pad 4: unconnected-(U8-V--Pad4) -> (no net)
- U8 pad 5: unconnected-(U8-NC-Pad5) -> (no net)
- U8 pad 6: unconnected-(U8-Pad6) -> (no net)
- U8 pad 7: unconnected-(U8-V+-Pad7) -> (no net)
- U8 pad 8: unconnected-(U8-NC-Pad8) -> (no net)
