File: Small_load_V1/Small_load_V1.kicad_pcb (KiCad board)
At the start: 2 copper layers, 101 x 101 mm, 110 parts, among them J1 USB_B, J10 Jack-DC, J11 Input, J3 Jack-DC, J4 Jack-DC, J5 Li ION cell own power, J6 Input, J8 INPUT, Q1 2N7002, Q10 IRFZ24NPBF, Q2 2N7002, Q3 IRFZ24NPBF, Q4 HYG025N06LS1C2, Q5 IRF9540N, Q6 HYG025N06LS1C2, Q7 2N3904, SW1 SW_SPST, SW3 RotaryEncoder_Switch, SW4 SW_SPST, U1 AD5337, U10 AD5337, U11 LM324A, U12 1602_LCD_I2C, U13 LM324A, U15 SRV05-4, U2 AD8001AR, U3 ESP32-S3-WROOM-1, U4 MCP3208, U5 CJ431, U6 LM5109BMA, U7 LM324A, U8 LM324A, U9 AD8001AR

Commit message: g
Parts:
- removed FID5: Polarity, Symbol:Polarity_Center_Positive_6mm_SilkScreen
- removed Q5: IRF9540N, Package_TO_SOT_THT:TO-220-3_Vertical
- added C13: 10u, Capacitor_SMD:C_1206_3216Metric, F.Cu at (341.8, 125.8)
- added C14: 10u, Capacitor_SMD:C_1206_3216Metric, F.Cu at (341.8, 129.2)
- added C15: 100n, Capacitor_SMD:C_0603_1608Metric, F.Cu at (275.1, 89.2)
- added C16: 1u, Capacitor_SMD:C_0402_1005Metric, F.Cu at (402.2, 104.5)
- added C17: 4n7, Capacitor_SMD:C_0402_1005Metric, F.Cu at (285.8, 82.9)
- added C18: 1u, Capacitor_SMD:C_0402_1005Metric, F.Cu at (285.8, 84.9)
- added C22: 100p, Capacitor_SMD:C_0603_1608Metric, F.Cu at (292.8, 67.6)
- added C23: 100n, Capacitor_SMD:C_0603_1608Metric, F.Cu at (252.7, 144.4)
- added C24: 10u, Capacitor_SMD:C_0603_1608Metric, F.Cu at (252.7, 146.9)
- added C25: 10u, Capacitor_SMD:C_0603_1608Metric, F.Cu at (252.7, 149.5)
- added C32: 4n7, Capacitor_SMD:C_0402_1005Metric, F.Cu at (402.2, 112.4)
- added C33: 1u, Capacitor_SMD:C_0402_1005Metric, F.Cu at (402.2, 114.4)
- added D6: LED_Small, LED_SMD:LED_0805_2012Metric, F.Cu at (261.4, 149.1)
- added D7: SS54, Diode_SMD:D_SMA, F.Cu at (275.1, 148.0)
- added J12: Conn_01x02, Z_mycustom_footprint_lib:MYOUNG MY-18650-01, F.Cu at (359.8, 36.4)
- added J7: Input, TerminalBlock:TerminalBlock_Altech_AK300-2_P5.00mm, F.Cu at (126.6, 54.2)
- added R33: 1k, Resistor_SMD:R_0603_1608Metric, F.Cu at (292.8, 80.1)
- added R34: 10k, Resistor_SMD:R_0603_1608Metric, F.Cu at (292.8, 82.6)
- added R35: 10k, Resistor_SMD:R_0603_1608Metric, F.Cu at (296.8, 67.6)
- added R36: 10k, Resistor_SMD:R_0603_1608Metric, F.Cu at (296.8, 70.1)
- added R37: 10k, Resistor_SMD:R_0603_1608Metric, F.Cu at (275.1, 91.7)
- added R38: 24k, Resistor_SMD:R_0603_1608Metric, F.Cu at (275.1, 94.2)
- added R39: 1k, Resistor_SMD:R_0603_1608Metric, F.Cu at (275.1, 96.7)
- added R40: 1k, Resistor_SMD:R_0603_1608Metric, F.Cu at (275.1, 99.2)
- added R42: 10k, Resistor_SMD:R_0603_1608Metric, F.Cu at (296.8, 75.1)
- added R43: 10k, Resistor_SMD:R_0603_1608Metric, F.Cu at (296.8, 77.6)
- added R44: 2.7M, Resistor_SMD:R_0603_1608Metric, F.Cu at (296.8, 80.1)
- added R45: 0R1, Resistor_SMD:R_1206_3216Metric, F.Cu at (360.2, 116.8)
- added R52: 1M, Resistor_SMD:R_0603_1608Metric, F.Cu at (300.8, 67.6)
- added R53: 10k, Resistor_SMD:R_0603_1608Metric, F.Cu at (300.8, 70.1)
- added R54: 56, Resistor_SMD:R_0603_1608Metric, F.Cu at (300.8, 72.6)
- added R55: 10k, Resistor_SMD:R_0603_1608Metric, F.Cu at (300.8, 75.1)
- added R56: 300, Resistor_SMD:R_0603_1608Metric_Pad0.98x0.95mm_HandSolder, F.Cu at (256.9, 144.4)
- added R57: 300, Resistor_SMD:R_0603_1608Metric_Pad0.98x0.95mm_HandSolder, F.Cu at (256.9, 146.9)
- added R58: 300, Resistor_SMD:R_0603_1608Metric_Pad0.98x0.95mm_HandSolder, F.Cu at (256.9, 149.5)
- added TP1: TestPoint, TestPoint:TestPoint_Pad_D1.0mm, F.Cu at (358.9, 112.1)
- added U14: INA219AxD, Package_SO:SOIC-8_3.9x4.9mm_P1.27mm, F.Cu at (396.6, 113.2)
- added U16: CH340C, Package_SO:SOIC-16_3.9x9.9mm_P1.27mm, F.Cu at (255.0, 137.5)
- added U17: AMS1117-3.3, Package_TO_SOT_SMD:SOT-223-3_TabPin2, F.Cu at (264.1, 135.9)
- C11: value 100p -> 100n
- D4: value 1N4007 -> SS54; footprint Diode_THT:D_DO-41_SOD81_P10.16mm_Horizontal -> Diode_SMD:D_SMA
- D5: value 1N4007 -> LED_Small; footprint Diode_THT:D_DO-41_SOD81_P10.16mm_Horizontal -> LED_SMD:LED_0805_2012Metric
- J5: value Li ION cell own power -> Input; footprint Z_mycustom_footprint_lib:MYOUNG MY-18650-01 -> TerminalBlock:TerminalBlock_Altech_AK300-2_P5.00mm
- Q7: value 2N3904 -> 2N7002; footprint Package_TO_SOT_THT:TO-92_Inline -> Package_TO_SOT_SMD:SOT-23
- R25: value 100 -> 50m; footprint Resistor_SMD:R_0603_1608Metric -> Resistor_THT:R_Axial_DIN0516_L15.5mm_D5.0mm_P20.32mm_Horizontal
- R26: value 1k -> 100
- R28: value 1k -> 0R1; footprint Resistor_SMD:R_0603_1608Metric -> Resistor_SMD:R_1206_3216Metric
- R29: value 10k -> 5R1; footprint Resistor_SMD:R_0603_1608Metric -> Resistor_SMD:R_0402_1005Metric
- R30: value 1k -> 5R1; footprint Resistor_SMD:R_0603_1608Metric -> Resistor_SMD:R_0402_1005Metric
- R32: value 10k -> 16k
- R41: value 50m -> 10k; footprint Resistor_THT:R_Axial_DIN0516_L15.5mm_D5.0mm_P20.32mm_Horizontal -> Resistor_SMD:R_0603_1608Metric
- R48: value 10k -> 0R1; footprint Resistor_SMD:R_0603_1608Metric -> Resistor_SMD:R_1206_3216Metric
- R49: value 40k2 -> 5R1; footprint Resistor_SMD:R_0603_1608Metric -> Resistor_SMD:R_0402_1005Metric
- R50: value 2k -> 5R1
- R51: value 10k -> 330k
- U11: value LM324A -> TPS5430DDAR; footprint Package_SO:SOIC-14_3.9x8.7mm_P1.27mm -> Package_SO:SOIC-8-1EP_3.9x4.9mm_P1.27mm_EP2.29x3mm_ThermalVias
- U13: value LM324A -> INA219AxD; footprint Package_SO:SOIC-14_3.9x8.7mm_P1.27mm -> Package_SO:SOIC-8_3.9x4.9mm_P1.27mm
- U2: value AD8001AR -> LM324; footprint Package_SO:SOIC-8_3.9x4.9mm_P1.27mm -> Package_SO:SOIC-14_3.9x8.7mm_P1.27mm
- U7: value LM324A -> LT3080xQ; footprint Package_SO:SOIC-14_3.9x8.7mm_P1.27mm -> Package_TO_SOT_SMD:TO-263-5_TabPin3
- U8: value LM324A -> LM324
- U9: value AD8001AR -> AD5337; footprint Package_SO:SOIC-8_3.9x4.9mm_P1.27mm -> Package_SO:MSOP-8_3x3mm_P0.65mm
- moved U12 216.2 mm to (68.8, 116.4), turned to 90 degrees
- moved R50 180.2 mm to (348.5, 117.5), turned to 0 degrees
- moved U9 176.3 mm to (353.7, 112.8), turned to 0 degrees
- moved R48 166.6 mm to (360.2, 120.0), turned to 0 degrees
- moved J1 163.4 mm to (66.2, 161.0), turned to 0 degrees
- moved J6 160.1 mm to (160.3, -19.3), turned to 180 degrees
- moved R49 157.4 mm to (348.5, 115.5), turned to 0 degrees
- moved U3 156.4 mm to (59.9, 137.3), turned to 90 degrees
- moved C12 153.6 mm to (158.0, 1.79)
- moved C8 153.6 mm to (158.0, -1.22)
- moved D2 153.6 mm to (173.0, 3.97)
- moved D3 153.6 mm to (173.0, 6.92)
- moved Q4 153.6 mm to (165.5, -4.03)
- moved Q6 153.6 mm to (171.9, -4.03)
- moved U6 153.6 mm to (166.6, 5.72)
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Connections:
- C11 pad 1: VLDO_OUT -> /LDO_Vcc
- C11 pad 2: Net-(U7B-+) -> GND
- C21 pad 1: +12V -> +5V
- C21 pad 2: -VDC -> GND
- C3 pad 2: Net-(U2--) -> Net-(U8A--)
- C56 pad 2: Net-(U9--) -> Net-(U8B--)
- D4 pad 1: GND -> /LDO_Vcc
- D5 pad 1: Net-(D4-A) -> Net-(D5-K)
- D5 pad 2: Net-(D5-A) -> +3V3
- J5 pad 1: +BATT -> GND
- J5 pad 2: GND -> Net-(J5-Pin_2)
- J6 pad 2: unconnected-(J6-Pin_2-Pad2) -> Net-(J6-Pin_2)
- Q7 pad 1: GND -> Net-(Q7-G)
- Q7 pad 2: Net-(Q7-B) -> GND
- Q7 pad 3: Net-(Q7-C) -> Net-(Q7-D)
- R1 pad 2: Net-(U2--) -> Net-(U8A--)
- R11 pad 1: Net-(Q5-S) -> Net-(U2C--)
- R11 pad 2: Net-(U7D--) -> GND
- R12 pad 1: /LDO_Vcc -> Net-(U2B-+)
- R12 pad 2: Net-(U7D-+) -> GND
- R2 pad 2: Net-(U9--) -> Net-(U8B--)
- R24 pad 1: Net-(Q7-B) -> Net-(U2C--)
- R24 pad 2: Net-(R24-Pad2) -> Net-(U7-SET)
- R25 pad 1: Net-(Q7-C) -> Net-(Q5-D)
- R25 pad 2: Net-(U13D-+) -> Net-(U7-IN)
- R26 pad 1: Net-(Q7-C) -> Net-(Q5-G)
- R28 pad 1: Net-(U11D--) -> /LDO_Vout
- R28 pad 2: GND -> Net-(D4-A)
- R29 pad 1: Net-(U11D--) -> Net-(D4-A)
- R29 pad 2: Net-(U13D-+) -> Net-(U13-IN+)
- R30 pad 1: Net-(U13D--) -> /LDO_Vout
- R30 pad 2: Net-(D5-A) -> Net-(U13-IN-)
- R32 pad 1: Net-(U13D--) -> Net-(U2D--)
- R32 pad 2: VLDO_OUT -> Net-(U7-IN)
- R41 pad 1: /LDO_Vcc -> SCL
- R41 pad 2: Net-(Q5-S) -> +3V3
- R46 pad 1: GND -> Net-(U2B-+)
- R46 pad 2: Net-(U7D-+) -> /LDO_Vcc
- R48 pad 1: Net-(U8D--) -> /CELL_CHARGER/Buck_out
- R48 pad 2: Net-(U7D--) -> Net-(J12-Pin_1)
- R49 pad 1: Net-(U7B-+) -> /CELL_CHARGER/Buck_out
- R49 pad 2: VLDO_OUT -> Net-(U14-IN+)
- R50 pad 1: GND -> Net-(J12-Pin_1)
- R50 pad 2: Net-(U7B-+) -> Net-(U14-IN-)
- R51 pad 1: Net-(Q5-G) -> Net-(Q7-D)
- R51 pad 2: Net-(Q5-S) -> Net-(U8C-+)
- R6 pad 2: Net-(U2--) -> Net-(U8A--)
- R7 pad 2: Net-(U9--) -> Net-(U8B--)
- U10 pad 8: GND -> +3V3
- U11 pad 1: (no net) -> Net-(U11-BOOT)
- U11 pad 2: (no net) -> unconnected-(U11-NC-Pad2)
- U11 pad 3: (no net) -> unconnected-(U11-NC-Pad3)
- U11 pad 4: (no net) -> Net-(U11-VSENSE)
- U11 pad 5: (no net) -> /BUCK_EN
- U11 pad 6: (no net) -> GND
- U11 pad 7: (no net) -> Net-(J5-Pin_2)
- U11 pad 8: (no net) -> Net-(D7-K)
- U11 pad 9: (no net) -> GND
- U13 pad 1: (no net) -> GND
- U13 pad 2: (no net) -> GND
- U13 pad 3: (no net) -> SDA
- U13 pad 4: (no net) -> SCL
- U13 pad 5: (no net) -> +3V3
- U13 pad 6: (no net) -> GND
- U13 pad 7: (no net) -> Net-(U13-IN-)
- U13 pad 8: (no net) -> Net-(U13-IN+)
- U2 pad 1: unconnected-(U2-NC-Pad1) -> Net-(U2A--)
- U2 pad 2: Net-(U2--) -> Net-(U2A--)
- U2 pad 3: /DAC1 -> GND
- U2 pad 4: unconnected-(U2-V--Pad4) -> /LDO_Vcc
- U2 pad 5: unconnected-(U2-NC-Pad5) -> Net-(U2B-+)
- U2 pad 6: Net-(C3-Pad1) -> /LDO_Vin
- U2 pad 7: unconnected-(U2-V+-Pad7) -> /LDO_Vin
- U2 pad 8: unconnected-(U2-NC-Pad8) -> Net-(U7-SET)
- U3 pad 13: D- -> unconnected-(U3-GPIO19/U1RTS/ADC2_CH8/CLK_OUT2/USB_D--Pad13)
- U3 pad 14: D+ -> unconnected-(U3-GPIO20/U1CTS/ADC2_CH9/CLK_OUT1/USB_D+-Pad14)
- U4 pad 10: unconnected-(U4-~{CS}/SHDN-Pad10) -> SPI_SS1
- U4 pad 11: unconnected-(U4-Din-Pad11) -> SPI_MOSI
- U4 pad 12: unconnected-(U4-Dout-Pad12) -> SPI_MISO
- U4 pad 13: unconnected-(U4-CLK-Pad13) -> SPI_clk
- U7 pad 1: (no net) -> unconnected-(U7-NC-Pad1)
- U7 pad 2: (no net) -> Net-(U7-SET)
- U7 pad 3: (no net) -> Net-(D4-A)
- U7 pad 4: (no net) -> Net-(U7-IN)
- U7 pad 5: (no net) -> Net-(U7-IN)
- U8 pad 1: (no net) -> Net-(C3-Pad1)
- U8 pad 10: (no net) -> Net-(U8C-+)
- U8 pad 11: (no net) -> GND
- U8 pad 12: /DAC3 -> Net-(Q3-S)
- U8 pad 13: Net-(U8D--) -> /Load_current_main
- U8 pad 14: Net-(R24-Pad2) -> /Load_current_main
- U8 pad 2: (no net) -> Net-(U8A--)
- U8 pad 3: (no net) -> /DAC1
- U8 pad 4: (no net) -> +5V
- U8 pad 5: (no net) -> /DAC2
- U8 pad 6: (no net) -> Net-(U8B--)
- U8 pad 7: (no net) -> Net-(C56-Pad1)
- U8 pad 8: (no net) -> /Load_voltage
- U8 pad 9: (no net) -> /Load_voltage
- U9 pad 1: unconnected-(U9-NC-Pad1) -> +3V3
- U9 pad 2: Net-(U9--) -> /CELL_CHARGER/DAC1
- U9 pad 3: /DAC2 -> /CELL_CHARGER/DAC2
- U9 pad 4: unconnected-(U9-V--Pad4) -> REF_2v5
- U9 pad 5: unconnected-(U9-NC-Pad5) -> GND
- U9 pad 6: Net-(C56-Pad1) -> SDA1
- U9 pad 7: unconnected-(U9-V+-Pad7) -> SCL1
- U9 pad 8: unconnected-(U9-NC-Pad8) -> GND
Other:
- board size 101 x 101 mm -> 101 x 121 mm
