File: Small_load_V1/CELL_CHARGER.kicad_sch (KiCad schematic)
At the start: 20 parts, among them J11 Conn_01x02, J7 Input, U11 AD5337, U11 TPS5430DDAR, U8 INA219AxD

Commit message: v
Parts:
- removed R25 (x2): 1k, Resistor_SMD:R_0603_1608Metric, symbol Device:R_Small
- added C27 (x2): 100u, Capacitor_THT:CP_Radial_D8.0mm_P3.50mm, symbol Device:C_Polarized_Small
- added C3: 100p, Capacitor_SMD:C_0402_1005Metric, symbol Device:C_Small
- added C34 (x3): 100n, Capacitor_SMD:C_0603_1608Metric, symbol Device:C_Small
- added C8: 10u@50V, Capacitor_SMD:C_0805_2012Metric, symbol Device:C
- added J9: connector, Connector_PinHeader_2.54mm:PinHeader_1x02_P2.54mm_Vertical, symbol Connector_Generic:Conn_01x02
- added R15: 100, Resistor_SMD:R_0603_1608Metric, symbol Device:R_Small
- added R8 (x2): 1k, Resistor_SMD:R_0603_1608Metric, symbol Device:R_Small
- J11: value Conn_01x02 -> 18650 holder
- L1: value L -> 75u; footprint (none) -> Inductor_SMD:L_Changjiang_FNR8040S
- R23, R64: value 5R1 -> 10
- R26: LCSC (none) -> C23352
Connections:
- net Buck_out: now also C27.1, C27.1, C3.1, C34.1, C34.1
- net GND: now also J11.1 (Pin_1), C27.2, C27.2, C34.2, C34.2, C34.2, C8.1, J9.1 (Pin_1), R8.2; no longer J11.2 (Pin_2)
- net Buck_SW: now reaches C7.2, D4.1 (K), L1.1, U11.8 (PH)
- net V_FB: now reaches R26.1, U11.4 (VSENSE)
- net V_FB: now also C3.2, R8.1, R8.1
- net at J7.2 (Pin_2), U11.7 (Vin): now also C34.1, C8.2
- net Boot_cap: now reaches C7.1, U11.1 (BOOT)
- net at R64.1, R72.2, R72.2: now also J11.2 (Pin_2), J9.2 (Pin_2); no longer J11.1 (Pin_1)
- net DAC1: no longer names the net of TP2.1, U11.2 (Vout_A)
- net DAC2 renamed DAC_cell
- net DAC_cell: now also R15.1
- new net: R15.2, R8.2
Other:
- note added: "+-26V max"
- note added: "1.221V Vsense"
- note added: "36V max"
- moved on the sheet: J7, L1
