File: Small_load_V1/buck.kicad_sch (KiCad schematic)
At the start: 16 parts, among them J11 Input, J14 Jack-DC, Q4 HYG025N06LS1C2, Q6 HYG025N06LS1C2, U6 LM5109BMA

Commit message: g
Parts:
- added C13, C14: 10u, Capacitor_SMD:C_1206_3216Metric, symbol Device:C_Small
- added L1: L, symbol Device:L
Connections:
- net GND: now also C13.2, C14.2
- net at C12.2, Q4.2 (S), Q6.1 (D)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: now also L1.1
- net at J11.2 (Pin_2): now also C13.1, C14.1, L1.2
Other:
- moved on the sheet: D3, J11, Q6, R21, R23

Commit message: v
Parts:
- added C27 (x2): 100u, Capacitor_THT:CP_Radial_D8.0mm_P3.50mm, symbol Device:C_Polarized_Small
- added C34: 100n, Capacitor_SMD:C_0603_1608Metric, symbol Device:C_Small
- added C42: 10u@50V, Capacitor_SMD:C_0805_2012Metric, symbol Device:C
- added J13, J9: jumper, Connector_PinHeader_2.54mm:PinHeader_1x02_P2.54mm_Vertical, symbol Connector_Generic:Conn_01x02
- added R12 (x2): 1k, Resistor_SMD:R_0603_1608Metric, symbol Device:R_Small
- added R34 (x3), R43 (x6): 10k, Resistor_SMD:R_0603_1608Metric, symbol Device:R_Small
- added R51 (x3): 100k, Resistor_SMD:R_0603_1608Metric, symbol Device:R_Small
- added R51: 330k, Resistor_SMD:R_0603_1608Metric, symbol Device:R_Small
- added R72: 0R1, Resistor_SMD:R_1206_3216Metric, symbol Device:R_Small
- added U18: LM317_TO-220, Package_TO_SOT_THT:TO-220-3_Vertical, symbol Regulator_Linear:LM317_TO-220
- added U19: LM324A, Package_SO:SOIC-14_3.9x8.7mm_P1.27mm, symbol Amplifier_Operational:LM324A
- L1: value L -> 75u; footprint (none) -> Inductor_SMD:L_Changjiang_FNR8040S
- R19, R20, R21, R23: value 56 -> 50; LCSC C25196 -> C23185
Connections:
- net +15V: now also C34.1, J13.2 (Pin_2)
- net GND: now also C27.2, C27.2, C34.2, C42.1, R12.2, R34.1, R34.1, R34.1, R43.1, R43.1, R43.1, R43.1, R43.1
- net Phase_A_H: now also R34.2
- net Phase_A_L: now also R34.2
- net buck_out: now reaches C13.1, C14.1, L1.2
- net buck_out: now also C27.1, R51.2, R72.1; no longer J11.2 (Pin_2)
- net buck_SW_node: now reaches C12.2, L1.1, Q4.2 (S), Q6.1 (D), U6.6 (HS)
- net at C10.1, C9.1, J14.1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: now also C27.1, J9.1 (Pin_1), R51.2
- new net: R43.2, R51.1, U19.3 (+)
- new net: C42.2, J13.1 (Pin_1), R12.1, U18.2 (VO)
- new net: R43.2, R51.1, U19.9 (-)
- new net: J11.2 (Pin_2), R51.2, R51.2, R72.2
- new net: J9.2 (Pin_2), R12.1, U18.3 (VI)
- new net: R43.2, R51.1, U19.10 (+)
- new net: R43.2, R51.1, U19.5 (+)
- new net: R12.2, R34.2, U18.1 (ADJ)
- new net SMPS_current: R43.1, U19.8
- new net SMPS_input: R43.2, U19.1, U19.2 (-)
- new net SMPS_output: R43.2, U19.6 (-), U19.7
Other:
- moved on the sheet: C10, C13, C14, C9, J11, J14
